File: avr_programmer/avr_programming_shield_Sockets.sch (EAGLE design)
At the start: 12 parts, among them IC1 ATMEGA168PROUND, IC2 TINY24/44/84-PU, U1 TINY85-20-DIP

Commit message: Added some text saying "DaveO was here to schematic view"
Other:
- note added: "Dave O was here - testing git"
Changed lines of the file:
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@@
 <?xml version="1.0" encoding="utf-8"?>
 <!DOCTYPE eagle SYSTEM "eagle.dtd">
-<eagle version="6.3">
+<eagle version="6.4">
 <drawing>
 <settings>
@@
 <text x="147.32" y="33.02" size="2.54" layer="94">AVR Programming Shield</text>
 <text x="147.32" y="27.94" size="2.54" layer="94">http://www.ladyada.net/make/mshield</text>
+<text x="30.48" y="25.4" size="1.778" layer="91">Dave O was here - testing git</text>
 </plain>
 <instances>
