File: avr_programmer/avr_programming_shield_built.sch (EAGLE design)
At the start: 19 parts

Commit message: updated bill of materials and adding uploaded build files
Parts:
- +PIEZO-, 16MHZ, ERR, HTB, ISP, ISP_328, ISP_84, ISP_85, JP2, JP4, MEGA_JUMPERS, PRG, R1, R2, R3, U$1, U$4: OC_NEWARK (none) -> unknown
- C1: MF (none) -> ILLINOIS CAPACITOR,INC.; MPN (none) -> 106TTA035M; OC_NEWARK (none) -> 30K6594
- RESET: MPN (none) -> B3F-1000; OC_NEWARK (none) -> 36M3542
Other:
- note added: "Bill Boucher Ken Olsen Dave Orth"
