File: avr_programmer/avr_programming_shield_v2b.brd (EAGLE design)
At the start: 47.6 x 53.3 mm, 22 parts

Commit message: update
Parts:
- removed E$1: (no value), adafruit:OSHWLOGO_TOL_0.2
- removed U$3: ZIFSOCKET-28-3ZIFFSOCKET-28-3, SparkFun:DIL28-3-ZIF_SOCKET
Routing:
- net VCC: track 40.3 -> 39.5 mm
- net RESET: track 36.2 -> 35.6 mm
Other:
- board text added: "."
- board text added: "MakersBox.blogspot.com"
- board text removed: "1"
- board text removed: "Burn bootloader"
- board text removed: "Insert target chip"
- board text removed: "Jumper ISP"
- board text removed: "Place ISP jumper"
- board text removed: "Tools -> Boards"
- board text removed: "Upload ArduinoISP"
- board text removed: "to target chip"
