File: osi/osi-blank.brd (EAGLE design)
At the start: 25.4 x 25.4 mm, 2 parts

Commit message: update
Parts:
- added CN1, CN2: 1X4-CLEANBIG, adafruit_mod:1X04-CLEANBIG
Connections:
- removed net D4: JP2.4
- removed net D6: JP2.2
- new net SCK: CN1.4, CN2.4, JP2.2
- new net SDA: CN1.3, CN2.3, JP2.4
- net GND: now also CN1.2, CN2.2
- net VCC: now also CN1.1, CN2.1
Other:
- outline, holes or cut-outs redrawn
Changed lines of the file:
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@@
 <setting verticaltext="up"/>
 </settings>
-<grid distance="0.025" unitdist="inch" unit="inch" style="lines" multiple="1" display="yes" altdistance="0.0001" altunitdist="inch" altunit="inch"/>
+<grid distance="0.05" unitdist="inch" unit="inch" style="lines" multiple="1" display="yes" altdistance="0.005" altunitdist="inch" altunit="inch"/>
 <layers>
 <layer number="1" name="Top" color="4" fill="1" visible="yes" active="yes"/>
@@
 <layer number="107" name="Crop" color="7" fill="1" visible="no" active="yes"/>
 <layer number="108" name="centerline" color="7" fill="1" visible="no" active="yes"/>
+<layer number="109" name="fp9" color="7" fill="1" visible="yes" active="yes"/>
+<layer number="110" name="fp0" color="7" fill="1" visible="yes" active="yes"/>
+<layer number="111" name="LPC17xx" color="7" fill="1" visible="yes" active="yes"/>
+<layer number="112" name="tSilk" color="7" fill="1" visible="yes" active="yes"/>
 <layer number="116" name="Patch_BOT" color="9" fill="4" visible="no" active="yes"/>
 <layer number="121" name="_tsilk" color="7" fill="1" visible="no" active="yes"/>
 <layer number="122" name="_bsilk" color="7" fill="1" visible="no" active="yes"/>
+<layer number="123" name="tTestmark" color="7" fill="1" visible="yes" active="yes"/>
+<layer number="124" name="bTestmark" color="7" fill="1" visible="yes" active="yes"/>
 <layer number="125" name="_tNames" color="7" fill="1" visible="no" active="yes"/>
+<layer number="126" name="_bNames" color="7" fill="1" visible="yes" active="yes"/>
+<layer number="127" name="_tValues" color="7" fill="1" visible="yes" active="yes"/>
+<layer number="128" name="_bValues" color="7" fill="1" visible="yes" active="yes"/>
 <layer number="131" name="prix" color="7" fill="1" visible="no" active="yes"/>
 <layer number="132" name="test" color="7" fill="1" visible="no" active="yes"/>
 <layer number="144" name="Drill_legend" color="7" fill="1" visible="no" active="yes"/>
 <layer number="151" name="HeatSink" color="7" fill="1" visible="no" active="yes"/>
+<layer number="152" name="_bDocu" color="7" fill="1" visible="yes" active="yes"/>
+<layer number="199" name="Contour" color="7" fill="1" visible="yes" active="yes"/>
 <layer number="200" name="200bmp" color="1" fill="10" visible="no" active="no"/>
 <layer number="201" name="201bmp" color="2" fill="10" visible="no" active="yes"/>
@@
 <layer number="223" name="223bmp" color="24" fill="1" visible="no" active="no"/>
 <layer number="224" name="224bmp" color="25" fill="1" visible="no" active="no"/>
+<layer number="248" name="Housing" color="7" fill="1" visible="yes" active="yes"/>
+<layer number="249" name="Edge" color="7" fill="1" visible="yes" active="yes"/>
 <layer number="250" name="Descript" color="3" fill="1" visible="no" active="no"/>
 <layer number="251" name="SMDround" color="12" fill="11" visible="no" active="no"/>
@@
 <board>
 <plain>
-<wire x1="0.635" y1="0" x2="24.767740625" y2="0" width="0" layer="20"/>
+<wire x1="1.905" y1="0" x2="24.767740625" y2="0" width="0" layer="20"/>
 <wire x1="24.767740625" y1="0" x2="24.767740625" y2="0.002740625" width="0" layer="20"/>
-<wire x1="24.767740625" y1="0.002740625" x2="25.4" y2="0.635" width="0" layer="20"/>
-<wire x1="25.4" y1="0.635" x2="25.4" y2="24.765" width="0" layer="20"/>
-<wire x1="25.4" y1="24.765" x2="24.7652" y2="25.3998" width="0" layer="20"/>
+<wire x1="24.767740625" y1="0.002740625" x2="25.4" y2="0" width="0" layer="20"/>
+<wire x1="25.4" y1="0" x2="25.4" y2="25.4" width="0" layer="20"/>
+<wire x1="25.4" y1="25.4" x2="24.7652" y2="25.3998" width="0" layer="20"/>
 <wire x1="24.7652" y1="25.3998" x2="24.7652" y2="25.4027" width="0" layer="20"/>
 <wire x1="24.7652" y1="25.4027" x2="0.635" y2="25.4" width="0" layer="20"/>
-<wire x1="0.635" y1="25.4" x2="0.000159375" y2="24.765159375" width="0" layer="20"/>
-<wire x1="0.000159375" y1="24.765159375" x2="0" y2="24.765159375" width="0" layer="20"/>
-<wire x1="0" y1="24.765159375" x2="0" y2="0.635" width="0" layer="20"/>
-<wire x1="0" y1="0.635" x2="0.635" y2="0" width="0" layer="20"/>
+<wire x1="0.635" y1="25.4" x2="0.000159375" y2="25.400159375" width="0" layer="20"/>
+<wire x1="0.000159375" y1="25.400159375" x2="0" y2="24.765159375" width="0" layer="20"/>
+<wire x1="0" y1="24.765159375" x2="0" y2="1.905" width="0" layer="20"/>
+<wire x1="0" y1="1.905" x2="1.905" y2="0" width="0" layer="20"/>
 <text x="19.685" y="8.89" size="1.016" layer="21" font="vector" ratio="10">RESET</text>
 <text x="0.70358125" y="2.7432" size="0.8128" layer="21" font="vector" ratio="15">VCC GND RST D8 D9 D10</text>
@@
 <element name="JP1" library="SparkFun_mod" package="1X06" value="" x="2.54" y="1.27"/>
 <element name="JP2" library="SparkFun_mod" package="1X08" value="" x="1.27" y="24.13"/>
+<element name="CN1" library="adafruit_mod" package="1X04-CLEANBIG" value="1X4-CLEANBIG" x="21.59" y="16.51" rot="R270"/>
+<element name="CN2" library="adafruit_mod" package="1X04-CLEANBIG" value="1X4-CLEANBIG" x="1.27" y="16.51" rot="R270"/>
 </elements>
 <signals>
@@
 <vertex x="-0.635" y="-0.635"/>
 </polygon>
+<contactref element="CN1" pad="2"/>
+<contactref element="CN2" pad="2"/>
+<wire x1="21.59" y1="17.78" x2="1.27" y2="17.78" width="0" layer="19" extent="1-1"/>
+<wire x1="5.08" y1="1.27" x2="21.59" y2="17.78" width="0" layer="19" extent="1-1"/>
 </signal>
 <signal name="VCC">
 <contactref element="JP1" pad="1"/>
+<contactref element="CN1" pad="1"/>
+<contactref element="CN2" pad="1"/>
+<wire x1="21.59" y1="20.32" x2="1.27" y2="20.32" width="0" layer="19" extent="1-1"/>
+<wire x1="2.54" y1="1.27" x2="21.59" y2="20.32" width="0" layer="19" extent="1-1"/>
 </signal>
 <signal name="RESET">
@@
 <contactref element="JP2" pad="1"/>
 </signal>
-<signal name="D4">
+<signal name="SDA">
 <contactref element="JP2" pad="4"/>
+<contactref element="CN1" pad="3"/>
+<contactref element="CN2" pad="3"/>
+<wire x1="21.59" y1="15.24" x2="8.89" y2="24.13" width="0" layer="19" extent="1-1"/>
+<wire x1="1.27" y1="15.24" x2="21.59" y2="15.24" width="0" layer="19" extent="1-1"/>
 </signal>
 <signal name="D3">
@@
 <contactref element="JP1" pad="4"/>
 </signal>
-<signal name="D6">
+<signal name="SCK">
 <contactref element="JP2" pad="2"/>
+<contactref element="CN1" pad="4"/>
+<contactref element="CN2" pad="4"/>
+<wire x1="21.59" y1="12.7" x2="3.81" y2="24.13" width="0" layer="19" extent="1-1"/>
+<wire x1="1.27" y1="12.7" x2="21.59" y2="12.7" width="0" layer="19" extent="1-1"/>
 </signal>
 </signals>
