File: osi/blank_rev_1.brd (EAGLE design)
At the start: 25.4 x 25.4 mm, 8 parts, among them IC1 TINY24/44/84-PU

Commit message: brain
Parts:
- removed C1: (no value), SparkFun:CAP-PTH-SMALL-KIT
- removed IC1: TINY24/44/84-PU, avr-7:DIL14
- removed JP5: M01PTH, SparkFun_mod:1X01
Connections:
- removed net D10: IC1.2, JP5.1
- net +3V3: no longer C1.2, IC1.1
- net AREF_D0: no longer IC1.13
- net D1: no longer IC1.12
- net D2: no longer IC1.11
- net D3: no longer IC1.10
- net D5: no longer IC1.8
- net D7: no longer IC1.6
- net D8: no longer IC1.5
- net D9: no longer IC1.3
- net GND: no longer C1.1, IC1.14
- net RESET: no longer IC1.4
- net SCL_D4: no longer IC1.9
- net SDA_D6: no longer IC1.7
Routing:
- net SDA_D6: track 42.8 -> 0.00 mm
- net +3V3: track 40.1 -> 0.00 mm
- net +5V: track 37.6 -> 0.00 mm
- net SCL_D4: track 35.9 -> 0.00 mm
- net AREF_D0: track 25.6 -> 0.00 mm
- net D1: track 20.9 -> 0.00 mm
- net D2: track 16.4 -> 0.00 mm
- net RESET: track 16.3 -> 0.00 mm
- net D8: track 16.1 -> 0.00 mm
- net D7: track 15.2 -> 0.00 mm
- net D3: track 12.6 -> 0.00 mm
- net D10: track 12.5 -> 0.00 mm
- net D9: track 9.94 -> 0.00 mm
- net D5: track 4.34 -> 0.00 mm

Commit message: power-ac
Parts:
- removed JP3: (no value), SparkFun_mod:1X06
- removed JP4: (no value), SparkFun_mod:1X08
- added JP5: (no value), SparkFun:1X06
- added JP6: (no value), SparkFun:1X08
Connections:
- net +3V3: now also JP5.4; no longer JP3.4
- net +5V: now also JP5.3; no longer JP3.3
- net AREF_D0: now also JP6.8; no longer JP4.8
- net D1: now also JP6.7; no longer JP4.7
- net D2: now also JP6.6; no longer JP4.6
- net D3: now also JP6.5; no longer JP4.5
- net D5: now also JP6.3; no longer JP4.3
- net D7: now also JP6.1; no longer JP4.1
- net D8: now also JP5.5; no longer JP3.5
- net D9: now also JP5.6; no longer JP3.6
- net GND: now also JP5.2; no longer JP3.2
- net SCL_D4: now also JP6.4; no longer JP4.4
- net SDA_D6: now also JP6.2; no longer JP4.2
- net V+: now also JP5.1; no longer JP3.1
Changed lines of the file:
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@@
 <setting verticaltext="up"/>
 </settings>
-<grid distance="0.025" unitdist="inch" unit="inch" style="lines" multiple="1" display="yes" altdistance="0.005" altunitdist="inch" altunit="inch"/>
+<grid distance="0.05" unitdist="inch" unit="inch" style="lines" multiple="1" display="yes" altdistance="0.005" altunitdist="inch" altunit="inch"/>
 <layers>
 <layer number="1" name="Top" color="4" fill="1" visible="yes" active="yes"/>
@@
 </autorouter>
 <elements>
-<element name="JP3" library="SparkFun_mod" package="1X06" value="" x="1.27" y="1.27"/>
-<element name="JP4" library="SparkFun_mod" package="1X08" value="" x="5.08" y="24.13"/>
 <element name="U$1" library="_my-parts" package="PTS635_SWITCH" value="PTS635_SWITCH" x="16.51" y="1.905"/>
 <element name="JP1" library="SparkFun_mod" package="1X05" value="" x="19.685" y="7.62" rot="R90"/>
 <element name="JP2" library="SparkFun_mod" package="1X05" value="" x="5.715" y="17.78" rot="R270"/>
+<element name="JP5" library="SparkFun" package="1X06" value="" x="1.27" y="1.27"/>
+<element name="JP6" library="SparkFun" package="1X08" value="" x="5.08" y="24.13"/>
 </elements>
 <signals>
@@
 </polygon>
 <contactref element="U$1" pad="P$1"/>
-<contactref element="JP3" pad="2"/>
 <contactref element="JP1" pad="3"/>
 <contactref element="JP2" pad="3"/>
+<contactref element="JP5" pad="2"/>
 <wire x1="16.51" y1="1.905" x2="19.685" y2="12.7" width="0" layer="19" extent="1-1"/>
+<wire x1="5.715" y1="12.7" x2="19.685" y2="12.7" width="0" layer="19" extent="1-1"/>
 <wire x1="3.81" y1="1.27" x2="16.51" y2="1.905" width="0" layer="19" extent="1-1"/>
-<wire x1="5.715" y1="12.7" x2="3.81" y2="1.27" width="0" layer="19" extent="1-1"/>
 </signal>
 <signal name="RESET">
 <contactref element="U$1" pad="P$2"/>
 </signal>
-<signal name="D3">
-<contactref element="JP4" pad="5"/>
-</signal>
-<signal name="D2">
-<contactref element="JP4" pad="6"/>
-</signal>
-<signal name="D1">
-<contactref element="JP4" pad="7"/>
-</signal>
-<signal name="AREF_D0">
-<contactref element="JP4" pad="8"/>
-</signal>
 <signal name="SDA_D6">
-<contactref element="JP4" pad="2"/>
 <contactref element="JP1" pad="2"/>
 <contactref element="JP2" pad="4"/>
-<wire x1="5.715" y1="10.16" x2="7.62" y2="24.13" width="0" layer="19" extent="1-1"/>
-<wire x1="19.685" y1="10.16" x2="5.715" y2="10.16" width="0" layer="19" extent="1-1"/>
-</signal>
-<signal name="V+">
-<contactref element="JP3" pad="1"/>
-</signal>
-<signal name="D5">
-<contactref element="JP4" pad="3"/>
+<contactref element="JP6" pad="2"/>
+<wire x1="5.715" y1="10.16" x2="19.685" y2="10.16" width="0" layer="19" extent="1-1"/>
+<wire x1="7.62" y1="24.13" x2="5.715" y2="10.16" width="0" layer="19" extent="1-1"/>
 </signal>
 <signal name="SCL_D4">
-<contactref element="JP4" pad="4"/>
 <contactref element="JP1" pad="1"/>
 <contactref element="JP2" pad="5"/>
-<wire x1="19.685" y1="7.62" x2="12.7" y2="24.13" width="0" layer="19" extent="1-1"/>
+<contactref element="JP6" pad="4"/>
 <wire x1="5.715" y1="7.62" x2="19.685" y2="7.62" width="0" layer="19" extent="1-1"/>
-</signal>
-<signal name="D8">
-<contactref element="JP3" pad="5"/>
-</signal>
-<signal name="D9">
-<contactref element="JP3" pad="6"/>
-</signal>
-<signal name="D7">
-<contactref element="JP4" pad="1"/>
+<wire x1="12.7" y1="24.13" x2="5.715" y2="7.62" width="0" layer="19" extent="1-1"/>
 </signal>
 <signal name="+3V3">
-<contactref element="JP3" pad="4"/>
 <contactref element="JP1" pad="4"/>
 <contactref element="JP2" pad="2"/>
+<contactref element="JP5" pad="4"/>
 <wire x1="5.715" y1="15.24" x2="19.685" y2="15.24" width="0" layer="19" extent="1-1"/>
 <wire x1="8.89" y1="1.27" x2="5.715" y2="15.24" width="0" layer="19" extent="1-1"/>
 </signal>
 <signal name="+5V">
-<contactref element="JP3" pad="3"/>
 <contactref element="JP1" pad="5"/>
 <contactref element="JP2" pad="1"/>
+<contactref element="JP5" pad="3"/>
 <wire x1="5.715" y1="17.78" x2="19.685" y2="17.78" width="0" layer="19" extent="1-1"/>
 <wire x1="6.35" y1="1.27" x2="5.715" y2="17.78" width="0" layer="19" extent="1-1"/>
 </signal>
+<signal name="D8">
+<contactref element="JP5" pad="5"/>
+</signal>
+<signal name="D9">
+<contactref element="JP5" pad="6"/>
+</signal>
+<signal name="V+">
+<contactref element="JP5" pad="1"/>
+</signal>
+<signal name="D3">
+<contactref element="JP6" pad="5"/>
+</signal>
+<signal name="D2">
+<contactref element="JP6" pad="6"/>
+</signal>
+<signal name="D1">
+<contactref element="JP6" pad="7"/>
+</signal>
+<signal name="AREF_D0">
+<contactref element="JP6" pad="8"/>
+</signal>
+<signal name="D5">
+<contactref element="JP6" pad="3"/>
+</signal>
+<signal name="D7">
+<contactref element="JP6" pad="1"/>
+</signal>
 </signals>
