File: osi/blank_rev_1.sch (EAGLE design)
At the start: 5 parts

Commit message: chuck
Parts:
- added R1, R2: (no value), adafruit_mod:R-US_0204/2V
Connections:
- removed net D8: JP6.5
- new net D10: JP6.6
- net D1: now also R2.2
- net D2: now also R1.2
- net D9: now also JP6.5; no longer JP6.6
- net GND: now also R1.1, R2.1
Changed lines of the file:
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@@
 <setting verticaltext="up"/>
 </settings>
-<grid distance="0.025" unitdist="inch" unit="inch" style="lines" multiple="1" display="no" altdistance="0.01" altunitdist="inch" altunit="inch"/>
+<grid distance="0.1" unitdist="inch" unit="inch" style="lines" multiple="1" display="no" altdistance="0.01" altunitdist="inch" altunit="inch"/>
 <layers>
 <layer number="1" name="Top" color="4" fill="1" visible="no" active="no"/>
@@
 <part name="JP8" library="SparkFun" deviceset="M08" device="1X08"/>
 <part name="FRAME1" library="SparkFun_mod" deviceset="FRAME-LETTER" device=""/>
+<part name="R1" library="adafruit_mod" deviceset="R-US_" device="0204/2V"/>
+<part name="R2" library="adafruit_mod" deviceset="R-US_" device="0204/2V"/>
+<part name="GND1" library="SparkFun" deviceset="GND" device=""/>
+<part name="GND3" library="SparkFun" deviceset="GND" device=""/>
 </parts>
 <sheets>
@@
 <instance part="FRAME1" gate="G$1" x="0" y="0"/>
 <instance part="FRAME1" gate="G$2" x="147.32" y="0"/>
+<instance part="R1" gate="G$1" x="177.8" y="63.5"/>
+<instance part="R2" gate="G$1" x="177.8" y="60.96"/>
+<instance part="GND1" gate="1" x="165.735" y="63.5" smashed="yes" rot="R270">
+<attribute name="VALUE" x="160.401" y="62.484" size="1.778" layer="96"/>
+</instance>
+<instance part="GND3" gate="1" x="165.735" y="60.96" smashed="yes" rot="R270">
+<attribute name="VALUE" x="160.401" y="59.944" size="1.778" layer="96"/>
+</instance>
 </instances>
 <busses>
@@
 <pinref part="JP6" gate="G$1" pin="2"/>
 </segment>
+<segment>
+<pinref part="R1" gate="G$1" pin="1"/>
+<pinref part="GND1" gate="1" pin="GND"/>
+<wire x1="168.275" y1="63.5" x2="172.72" y2="63.5" width="0.1524" layer="91"/>
+</segment>
+<segment>
+<pinref part="R2" gate="G$1" pin="1"/>
+<pinref part="GND3" gate="1" pin="GND"/>
+<wire x1="168.275" y1="60.96" x2="172.72" y2="60.96" width="0.1524" layer="91"/>
+</segment>
 </net>
 <net name="RESET" class="0">
@@
 <net name="D2" class="0">
 <segment>
-<wire x1="191.135" y1="63.5" x2="183.515" y2="63.5" width="0.1524" layer="91"/>
+<wire x1="191.135" y1="63.5" x2="182.88" y2="63.5" width="0.1524" layer="91"/>
 <pinref part="JP8" gate="G$1" pin="6"/>
 <label x="187.325" y="63.5" size="1.778" layer="95"/>
+<pinref part="R1" gate="G$1" pin="2"/>
 </segment>
 </net>
 <net name="D1" class="0">
 <segment>
-<wire x1="191.135" y1="60.96" x2="183.515" y2="60.96" width="0.1524" layer="91"/>
+<wire x1="191.135" y1="60.96" x2="182.88" y2="60.96" width="0.1524" layer="91"/>
 <pinref part="JP8" gate="G$1" pin="7"/>
 <label x="187.325" y="60.96" size="1.778" layer="95"/>
+<pinref part="R2" gate="G$1" pin="2"/>
 </segment>
 </net>
@@
 </segment>
 </net>
-<net name="D8" class="0">
+<net name="D9" class="0">
 <segment>
 <wire x1="160.655" y1="86.36" x2="191.135" y2="86.36" width="0.1524" layer="91"/>
@@
 </segment>
 </net>
-<net name="D9" class="0">
+<net name="D10" class="0">
 <segment>
 <wire x1="160.655" y1="83.82" x2="191.135" y2="83.82" width="0.1524" layer="91"/>

Commit message: D9 -> D8 for INT0
Connections:
- net D9 renamed D8
Changed lines of the file:
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@@
 </segment>
 </net>
-<net name="D9" class="0">
+<net name="D8" class="0">
 <segment>
 <wire x1="160.655" y1="86.36" x2="191.135" y2="86.36" width="0.1524" layer="91"/>
