File: osi/blank_rev_2.brd (EAGLE design)
At the start: 25.4 x 25.4 mm, 8 parts

Commit message: layout changes
Parts:
- removed I2C_L, I2C_R: (no value), SparkFun_mod:1X05
- removed JP8: (no value), SparkFun:1X08
- removed R1, R2: (no value), adafruit_mod:0204V
- removed RESET: PTS635_SWITCH, _my-parts:PTS635_SWITCH
- removed U$1: AVR-MEGA8-AI, SparkFun:TQFP32-08
- added JP5: (no value), SparkFun_mod:1X08
- moved JP6 1.80 mm to (2.54, 2.54)
Connections:
- removed net AREF_D0: JP8.8
- removed net D1: JP8.7, R2.2
- removed net D10: JP6.6
- removed net D2: JP8.6, R1.2
- removed net D3: JP8.5
- removed net D5: JP8.3
- removed net D7: JP8.1
- removed net D8: JP6.5
- removed net SCL_D4: I2C_L.1, I2C_R.5, JP8.4
- removed net SDA_D6: I2C_L.2, I2C_R.4, JP8.2
- new net A0: JP5.2
- new net A1: JP5.1
- new net A2: JP6.1
- new net A3: JP6.2
- new net A6: JP6.3
- new net A7: JP5.3
- new net D11: JP5.6
- new net D12: JP5.5
- new net D13: JP5.4
- net +3V3: no longer I2C_L.4, I2C_R.2
- net +5V: now also JP5.7; no longer I2C_L.5, I2C_R.1, JP6.3
- net GND: now also JP6.5; no longer I2C_L.3, I2C_R.3, JP6.2, R1.1, R2.1, RESET.P$1
- net RESET: now also JP6.6; no longer RESET.P$2
- net V+: now also JP5.8; no longer JP6.1
Other:
- outline, holes or cut-outs redrawn
- board text added: "11"
- board text added: "12"
- board text added: "13"
- board text added: "A0"
- board text added: "A1"
- board text added: "A2"
- board text added: "A3"
- board text added: "A6"
- board text added: "A7"
- board text added: "Apr 12"
- board text added: "Atmega328"
- board text added: "D11"
- board text added: "D12"
- board text added: "D13"
- board text added: "NODE"
- board text added: "RST"
- board text added: "i2c"
- board text removed: "+5V"
- board text removed: "3V3"
- board text removed: "BRAIN"
- board text removed: "Brain Rev 1 Feb 12"
- board text removed: "D0"
- board text removed: "D1"
- board text removed: "D10"
- board text removed: "D2"
- board text removed: "D3"
- board text removed: "D4"
- board text removed: "D5"
- board text removed: "D6"
- board text removed: "D7"
- board text removed: "D9"
- board text removed: "One Square Inch"
- board text removed: "RESET"
- board text removed: "SCK"
- board text removed: "SDA"
