File: osi/blank_rev_3dip.brd (EAGLE design)
At the start: 50.8 x 27.9 mm, 20 parts, among them IC2 ATMEGA168-20P, Y2 8Mhz

Commit message: double board finished?
Parts:
- added JP7: (no value), SparkFun_mod:1X02
- added U$1: (no value), _my-parts:OREGON_24_52
- added U$2: (no value), _my-parts:OREGON_24_51
- moved JP9 11.4 mm to (39.4, 3.81)
- moved R3 11.3 mm to (28.6, 7.62), turned to 0 degrees
- moved Y2 2.54 mm to (29.2, 4.45)
- moved C2 1.91 mm to (43.2, 21.6), turned to 180 degrees
- moved R2 1.42 mm to (34.3, 21.6), turned to 180 degrees
- moved R1 1.42 mm to (38.1, 7.62)
- moved JP12 1.27 mm to (6.35, 19.1)
- moved JP2 1.27 mm to (6.35, 6.35)
- moved JP3 1.27 mm to (44.5, 6.35)
- moved JP4 1.27 mm to (44.5, 19.1)
- moved S1 0.25 mm to (21.0, 3.30), turned to 180 degrees
Connections:
- net GND: now also S1.3, S1.4; no longer S1.1, S1.2
- net RESET: now also S1.1, S1.2; no longer S1.3, S1.4
- net SCL_A5: now also JP7.2
- net SDA_A4: now also JP7.1
Routing:
- net +3V3: track 100.1 -> 153.7 mm
- net A0: track 0.00 -> 30.4 mm
- net A1: track 0.00 -> 29.7 mm
- net D8: track 0.00 -> 23.3 mm
- net D13: track 0.00 -> 20.5 mm
- net D12: track 0.00 -> 17.6 mm
- net SDA_A4: track 84.6 -> 69.3 mm
- net RESET: track 80.9 -> 66.8 mm
- net D10: track 23.1 -> 18.1 mm
- net SCL_A5: track 73.6 -> 78.6 mm
- net +5V: track 110.4 -> 115.1 mm
- net V+: track 116.1 -> 119.9 mm
- net N$1: track 3.17 -> 6.77 mm
- net D9: track 22.4 -> 19.2 mm
- net N$4: track 0.00 -> 2.54 mm
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Other:
- outline, holes or cut-outs redrawn
- board text added: "Atmega328"
- board text added: "D13"
- board text added: "DTR"
- board text removed: "A6"
- board text removed: "A7"
