File: osi/blank_rev_3dip.sch (EAGLE design)
At the start: 20 parts, among them IC2 ATMEGA168-20P, Y2 8Mhz

Commit message: double board finished?
Parts:
- added JP7: (no value), SparkFun_mod:M02PTH
Connections:
- net GND: now also S1.3, S1.4; no longer S1.1, S1.2
- net RESET: now also S1.1, S1.2; no longer S1.3, S1.4
- net SCL_A5: now also JP7.2
- net SDA_A4: now also JP7.1
Changed lines of the file:
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@@
 <part name="JP12" library="SparkFun_mod" deviceset="M02" device="PTH"/>
 <part name="GND7" library="SparkFun" deviceset="GND" device=""/>
+<part name="JP7" library="SparkFun_mod" deviceset="M02" device="PTH"/>
 </parts>
 <sheets>
@@
 <instance part="C1" gate="G$1" x="-38.1" y="86.36"/>
 <instance part="C2" gate="G$1" x="-38.1" y="58.42"/>
-<instance part="S1" gate="S" x="-48.26" y="76.2"/>
+<instance part="S1" gate="S" x="-48.26" y="76.2" rot="MR0"/>
 <instance part="LED1" gate="G$1" x="53.34" y="5.08" rot="R270"/>
 <instance part="R4" gate="G$1" x="43.18" y="5.08" rot="R180"/>
@@
 <instance part="JP12" gate="G$1" x="5.08" y="139.7" rot="R180"/>
 <instance part="GND7" gate="1" x="-20.32" y="66.04" rot="R270"/>
+<instance part="JP7" gate="G$1" x="55.88" y="109.22" rot="R180"/>
 </instances>
 <busses>
@@
 </segment>
 <segment>
-<pinref part="GND3" gate="1" pin="GND"/>
-<wire x1="-55.88" y1="76.2" x2="-53.34" y2="76.2" width="0.1524" layer="91"/>
-<pinref part="S1" gate="S" pin="1"/>
-<pinref part="S1" gate="S" pin="2"/>
-<wire x1="-53.34" y1="76.2" x2="-53.34" y2="73.66" width="0.1524" layer="91"/>
-<junction x="-53.34" y="76.2"/>
-</segment>
-<segment>
 <pinref part="R4" gate="G$1" pin="2"/>
 <pinref part="GND6" gate="1" pin="GND"/>
@@
 <wire x1="-10.16" y1="66.04" x2="-17.78" y2="66.04" width="0.1524" layer="91"/>
 <pinref part="GND7" gate="1" pin="GND"/>
+</segment>
+<segment>
+<pinref part="GND3" gate="1" pin="GND"/>
+<wire x1="-55.88" y1="76.2" x2="-55.88" y2="73.66" width="0.1524" layer="91"/>
+<pinref part="S1" gate="S" pin="4"/>
+<wire x1="-55.88" y1="73.66" x2="-53.34" y2="73.66" width="0.1524" layer="91"/>
+<pinref part="S1" gate="S" pin="3"/>
+<wire x1="-55.88" y1="76.2" x2="-53.34" y2="76.2" width="0.1524" layer="91"/>
+<junction x="-55.88" y="76.2"/>
 </segment>
 </net>
@@
 <wire x1="99.06" y1="76.2" x2="-30.48" y2="76.2" width="0.1524" layer="91"/>
 <wire x1="-30.48" y1="76.2" x2="-38.1" y2="76.2" width="0.1524" layer="91"/>
-<wire x1="-38.1" y1="76.2" x2="-43.18" y2="76.2" width="0.1524" layer="91"/>
 <junction x="-38.1" y="81.28"/>
 <wire x1="-10.16" y1="71.12" x2="-30.48" y2="71.12" width="0.1524" layer="91"/>
 <wire x1="-30.48" y1="71.12" x2="-30.48" y2="76.2" width="0.1524" layer="91"/>
 <junction x="-30.48" y="76.2"/>
-<wire x1="-43.18" y1="73.66" x2="-43.18" y2="76.2" width="0.1524" layer="91"/>
 <pinref part="R2" gate="G$1" pin="2"/>
 <pinref part="C1" gate="G$1" pin="2"/>
-<pinref part="S1" gate="S" pin="3"/>
-<junction x="-43.18" y="76.2"/>
-<pinref part="S1" gate="S" pin="4"/>
 <wire x1="99.06" y1="76.2" x2="99.06" y2="109.22" width="0.1524" layer="91"/>
 <label x="119.38" y="109.22" size="1.778" layer="95"/>
@@
 <wire x1="-38.1" y1="81.28" x2="-38.1" y2="76.2" width="0.1524" layer="91"/>
 <pinref part="IC2" gate="G$1" pin="PC6(/RESET/PCI14)"/>
+<wire x1="-40.64" y1="73.66" x2="-40.64" y2="76.2" width="0.1524" layer="91"/>
+<wire x1="-40.64" y1="76.2" x2="-38.1" y2="76.2" width="0.1524" layer="91"/>
+<junction x="-38.1" y="76.2"/>
+<pinref part="S1" gate="S" pin="2"/>
+<wire x1="-40.64" y1="73.66" x2="-43.18" y2="73.66" width="0.1524" layer="91"/>
+<pinref part="S1" gate="S" pin="1"/>
+<wire x1="-43.18" y1="76.2" x2="-40.64" y2="76.2" width="0.1524" layer="91"/>
+<junction x="-40.64" y="76.2"/>
 </segment>
 </net>
@@
 <label x="43.18" y="119.38" size="1.778" layer="95"/>
 </segment>
+<segment>
+<pinref part="JP7" gate="G$1" pin="1"/>
+<wire x1="48.26" y1="109.22" x2="43.18" y2="109.22" width="0.1524" layer="91"/>
+<label x="43.18" y="109.22" size="1.778" layer="95"/>
+</segment>
 </net>
 <net name="SCL_A5" class="0">
@@
 <label x="43.18" y="116.84" size="1.778" layer="95"/>
 </segment>
-</net>
+<segment>
+<pinref part="JP7" gate="G$1" pin="2"/>
+<wire x1="48.26" y1="106.68" x2="43.18" y2="106.68" width="0.1524" layer="91"/>
+<label x="43.18" y="106.68" size="1.778" layer="95"/>
+</segment>
+</net>
