File: osi/brain/osi-brain_rev_1.brd (EAGLE design)
At the start: 25.4 x 25.4 mm, 8 parts, among them IC1 TINY24/44/84-PU

Commit message: power-ac
Parts:
- JP3: device SparkFun_mod:1X06 -> SparkFun:1X06
- JP4: device SparkFun_mod:1X08 -> SparkFun:1X08
- JP5: value M01PTH -> (none); device SparkFun_mod:1X01 -> SparkFun_mod:1X02_NO_SILK
- moved JP5 0.63 mm to (5.71, 5.08), turned to 180 degrees
Connections:
- net GND: now also JP5.2
Routing:
- net +5V: track 37.6 -> 39.2 mm
- net D10: track 12.5 -> 11.8 mm
