File: osi/brain/brain_rev_101.sch (EAGLE design)
At the start: 10 parts, among them IC1 TINY24/44/84-PU

Commit message: continue on brain
Connections:
- removed net D10: IC1.(PCINT8/XTAL1/CLKI)PB0, JP6.6
- net RESET: now also JP6.6
Changed lines of the file:
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@@
 <wire x1="88.9" y1="78.74" x2="78.74" y2="78.74" width="0.1524" layer="91"/>
 <pinref part="U$1" gate="G$1" pin="P$2"/>
+<wire x1="88.9" y1="63.5" x2="99.06" y2="63.5" width="0.1524" layer="91"/>
+<junction x="88.9" y="63.5"/>
+<wire x1="99.06" y1="63.5" x2="99.06" y2="55.88" width="0.1524" layer="91"/>
+<pinref part="JP6" gate="G$1" pin="6"/>
+<wire x1="99.06" y1="55.88" x2="121.92" y2="55.88" width="0.1524" layer="91"/>
 </segment>
 </net>
@@
 </segment>
 </net>
-<net name="D10" class="0">
-<segment>
-<pinref part="IC1" gate="1" pin="(PCINT8/XTAL1/CLKI)PB0"/>
-<label x="121.539" y="57.785" size="1.778" layer="95" rot="R180"/>
-<pinref part="JP6" gate="G$1" pin="6"/>
-<wire x1="88.9" y1="55.88" x2="121.92" y2="55.88" width="0.1524" layer="91"/>
-</segment>
-</net>

Commit message: Programming shield ver 1.2
Parts:
- removed IC2_L, IC2_R: (no value), SparkFun_mod:M05PTH
- removed JP8: (no value), SparkFun:M081X08
- added J1: AVR_SPI_PRG_6PTH, SparkFun_mod:AVR_SPI_PRG_6PTH
- added JP1, JP2: (no value), SparkFun_mod:M04PTH
- added JP3, JP4: (no value), SparkFun_mod:M02PTH
- added JP5: (no value), SparkFun_mod:M081X08
Connections:
- net +3V3: now also JP1.1, JP2.4; no longer IC2_L.4, IC2_R.2
- net +5V: now also JP3.2, JP4.1; no longer IC2_L.5, IC2_R.1
- net AREF_D0: now also JP5.8; no longer JP8.8
- net D1: now also JP5.7; no longer JP8.7
- net D2: now also JP5.6; no longer JP8.6
- net D3: now also JP5.5; no longer JP8.5
- net D5: now also JP5.3; no longer JP8.3
- net D7: now also JP5.1; no longer JP8.1
- net GND: now also JP1.2, JP2.3; no longer IC2_L.3, IC2_R.3
- net SCL_D4: now also JP1.4, JP2.1, JP5.4; no longer IC2_L.1, IC2_R.5, JP8.4
- net SDA_D6: now also JP1.3, JP2.2, JP5.2; no longer IC2_L.2, IC2_R.4, JP8.2
- net V+: now also JP3.1, JP4.2
