File: osi/brain/brain_rev_103.brd (EAGLE design)
At the start: 25.4 x 25.4 mm, 8 parts

Commit message: 328 TFOP?
Parts:
- removed I2C_L, I2C_R: (no value), SparkFun_mod:1X05
- removed JP8: (no value), SparkFun:1X08
- removed R1: (no value), adafruit_mod:0204V
- removed RESET: PTS635_SWITCH, _my-parts:PTS635_SWITCH
- added C1, C2: (no value), SparkFun:CAP-PTH-SMALL-KIT
- added JP2: (no value), SparkFun_mod:1X04
- added JP3: (no value), SparkFun_mod:1X02
- added JP5: (no value), SparkFun_mod:1X08
- added JP7: FTDI Basic, SparkFun:1X06
- added R3, R4: (no value), adafruit_mod:0204V
- added U1: ATMEGA168, SparkFun:TQFP32-08
- U$1: value AVR-MEGA8-AI -> PTS635_SWITCH; device SparkFun:TQFP32-08 -> _my-parts:PTS635_SWITCH
- moved R2 33.8 mm to (15.4, 20.6)
- moved U$1 16.0 mm to (23.1, 1.78), turned to 180 degrees
Connections:
- removed net AREF_D0: JP8.8
- removed net D1: JP8.7, R2.2
- removed net D2: JP8.6, R1.2
- removed net D3: JP8.5
- removed net D5: JP8.3
- removed net D7: JP8.1
- removed net D8: JP6.5
- removed net SCL_D4: I2C_L.1, I2C_R.5, JP8.4
- removed net SDA_D6: I2C_L.2, I2C_R.4, JP8.2
- new net A0: JP5.4, U1.23
- new net A1: JP5.3, U1.24
- new net A2: JP5.2, U1.25
- new net A3: JP5.1, U1.26
- new net D11: JP5.7, U1.15
- new net D12: JP5.6, U1.16
- new net D13: JP5.5, U1.17
- new net D9: JP6.5, U1.13
- new net DTR: C2.2, JP7.1
- new net RXI: JP7.3, U1.30
- new net SCL_A5: JP2.1, R3.2, U1.28
- new net SDA_A4: JP2.2, R2.2, U1.27
- new net TXO: JP7.2, U1.31
- net +3V3: now also C1.2, JP2.4, JP7.4, R2.1, R3.1, R4.1, U1.18, U1.20, U1.4, U1.6; no longer I2C_L.4, I2C_R.2
- net +5V: now also JP3.2; no longer I2C_L.5, I2C_R.1
- net D10: now also JP5.8, U1.14; no longer JP6.6
- net GND: now also C1.1, JP2.3, JP7.5, JP7.6, U$1.P$1, U1.21, U1.3, U1.5; no longer I2C_L.3, I2C_R.3, R1.1, R2.1, RESET.P$1
- net RESET: now also C2.1, JP6.6, R4.2, U$1.P$2, U1.29; no longer RESET.P$2
- net V+: now also JP3.1
Routing:
- net SCL_A5: track 0.00 -> 46.7 mm, vias 0 -> 1
- net +3V3: track 0.00 -> 41.9 mm, vias 0 -> 1
- net SDA_A4: track 0.00 -> 31.8 mm, vias 0 -> 1
- net +5V: track 0.00 -> 28.3 mm
- net D9: track 0.00 -> 24.9 mm, vias 0 -> 1
- net V+: track 0.00 -> 16.8 mm
- net D10: track 0.00 -> 14.4 mm
- net A3: track 0.00 -> 12.0 mm
- net D11: track 0.00 -> 11.6 mm
- net A2: track 0.00 -> 11.2 mm
- net TXO: track 0.00 -> 10.8 mm
- net RESET: track 0.00 -> 10.5 mm
- net D12: track 0.00 -> 9.31 mm
- net A0: track 0.00 -> 8.86 mm
- net A1: track 0.00 -> 8.44 mm
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Other:
- outline, holes or cut-outs redrawn
- board text added: "A0"
- board text added: "A1"
- board text added: "A2"
- board text added: "A3"
- board text added: "A4"
- board text added: "Apr 12"
- board text added: "D11"
- board text added: "D12"
- board text added: "D13"
- board text added: "NODE"
- board text added: "RST"
- board text added: "Vin"
- board text removed: "+5V"
- board text removed: "BRAIN"
- board text removed: "Brain Rev 1 Feb 12"
- board text removed: "D0"
- board text removed: "D1"
- board text removed: "D2"
- board text removed: "D3"
- board text removed: "D4"
- board text removed: "D5"
- board text removed: "D6"
- board text removed: "D7"
- board text removed: "One Square Inch"
