File: osi/brain/brain_rev_103.sch (EAGLE design)
At the start: 8 parts

Commit message: 328 TFOP?
Parts:
- removed I2C_L, I2C_R: (no value), SparkFun_mod:M05PTH
- removed JP8: (no value), SparkFun:M081X08
- removed R1: (no value), adafruit_mod:R-US_0204/2V
- removed RESET: PTS635_SWITCH, _my-parts:PTS635_SWITCH
- added C1, C2: (no value), SparkFun:CAPKIT
- added JP2: (no value), SparkFun_mod:M04PTH
- added JP3: (no value), SparkFun_mod:M02PTH
- added JP5: (no value), SparkFun_mod:M081X08
- added JP7: FTDI Basic, SparkFun:ARDUINO_SERIAL_PROGRAMPTH
- added R3, R4: (no value), adafruit_mod:R-US_0204/2V
- added U1: ATMEGA168, SparkFun:ATMEGA168
- U$1: value AVR-MEGA8-AI -> PTS635_SWITCH; device SparkFun:AVR-MEGA8-AI -> _my-parts:PTS635_SWITCH
Connections:
- removed net AREF_D0: JP8.8
- removed net D1: JP8.7, R2.2
- removed net D2: JP8.6, R1.2
- removed net D3: JP8.5
- removed net D5: JP8.3
- removed net D7: JP8.1
- removed net D8: JP6.5
- removed net SCL_D4: I2C_L.1, I2C_R.5, JP8.4
- removed net SDA_D6: I2C_L.2, I2C_R.4, JP8.2
- new net A0: JP5.4, U1.PC0(ADC0)
- new net A1: JP5.3, U1.PC1(ADC1)
- new net A2: JP5.2, U1.PC2(ADC2)
- new net A3: JP5.1, U1.PC3(ADC3)
- new net D11: JP5.7, U1.PB3(MOSI/OC2)
- new net D12: JP5.6, U1.PB4(MISO)
- new net D13: JP5.5, U1.PB5(SCK)
- new net D9: JP6.5, U1.PB1(OC1A)
- new net DTR: C2.2, JP7.DTR
- new net RXI: JP7.TXO, U1.PD0(RXD)
- new net SCL_A5: JP2.1, R3.2, U1.PC5(ADC5/SCL)
- new net SDA_A4: JP2.2, R2.2, U1.PC4(ADC4/SDA)
- new net TXO: JP7.RXI, U1.PD1(TXD)
- net +3V3: now also C1.2, JP2.4, JP7.VCC, R2.1, R3.1, R4.1, U1.AREF, U1.AVCC, U1.VCC@1, U1.VCC@2; no longer I2C_L.4, I2C_R.2
- net +5V: now also JP3.2; no longer I2C_L.5, I2C_R.1
- net D10: now also JP5.8, U1.PB2(SS/OC1B); no longer JP6.6
- net GND: now also C1.1, JP2.3, JP7.CTS, JP7.GND, U$1.P$1, U1.AGND, U1.GND@1, U1.GND@2; no longer I2C_L.3, I2C_R.3, R1.1, R2.1, RESET.P$1
- net RESET: now also C2.1, JP6.6, R4.2, U$1.P$2, U1.PC6(/RESET); no longer RESET.P$2
- net V+: now also JP3.1
Other:
- moved on the sheet: JP6, R2
