File: osi/brain/brain_rev_2.brd (EAGLE design)
At the start: 25.4 x 25.4 mm, 15 parts, among them U1 ATMEGA168, Y1 RESONATORSMD

Commit message: layout changes
Parts:
- removed S1: (no value), SparkFun:TACTILE_SWITCH_SMD
- added SW1: SPST_TACT-KMR2, adafruit:KMR2
- added U$1: (no value), adafruit:OSHWLOGO_TOL_0.2
- moved LED1 12.2 mm to (18.4, 2.86), turned to 180 degrees
- moved R1 10.1 mm to (13.6, 5.33), turned to 180 degrees
- moved R2 5.24 mm to (18.7, 6.67), turned to 0 degrees
- moved R4 2.16 mm to (18.7, 10.9)
- moved R3 2.16 mm to (18.7, 8.76)
Connections:
- net A6: now also JP6.3
- net D10: no longer JP6.3
- net GND: now also SW1.1; no longer S1.2
- net RESET: now also SW1.2, SW1.4; no longer S1.3
Routing:
- net A6: track 0.00 -> 21.2 mm, vias 0 -> 1
- net D10: track 19.4 -> 0.00 mm, vias 1 -> 0
- net RESET: track 48.2 -> 59.4 mm, vias 0 -> 1
- net D3: track 3.37 -> 13.4 mm, vias 0 -> 2
- net N$4: track 2.22 -> 5.90 mm
- net +3V3: track 101.8 -> 99.9 mm
- net SCL_A5: track 24.2 -> 24.9 mm
- net SDA_A4: track 23.1 -> 23.9 mm
Other:
- board text added: "A6"
- board text removed: "10"
- board text removed: "D10"

Commit message: Furby
Parts:
- removed JP5: (no value), SparkFun_mod:1X08
- added JP1: (no value), SparkFun:1X08
- U$1: device adafruit:OSHWLOGO_TOL_0.2 -> adafruit_mod:OSHWLOGO_BOTTOM
- moved U$1 12.7 mm to (17.8, 15.7)
- moved R4 3.30 mm to (19.6, 14.1), turned to 90 degrees
- moved R3 1.52 mm to (18.7, 10.3)
- moved Y1 0.76 mm to (13.7, 8.13)
- moved R2 0.76 mm to (18.7, 7.43)
- moved R1 0.25 mm to (13.3, 5.33)
Connections:
- net +5V: now also JP1.7; no longer JP5.7
- net A0: now also JP1.2; no longer JP5.2
- net A1: now also JP1.1; no longer JP5.1
- net A7: now also JP1.3; no longer JP5.3
- net D11: now also JP1.6; no longer JP5.6
- net D12: now also JP1.5; no longer JP5.5
- net D13: now also JP1.4; no longer JP5.4
- net V+: now also JP1.8; no longer JP5.8
Routing:
- net SDA_A4: track 23.9 -> 26.1 mm
- net SCL_A5: track 24.9 -> 26.0 mm
- net +3V3: track 99.9 -> 100.7 mm
- net RESET: track 59.4 -> 60.1 mm
- net N$3: track 3.47 -> 4.09 mm
Other:
- board text added: "Open Source Hardware"
- board text added: "Rev 2 Apr 12"
- board text removed: "Apr 12"
