File: osi/brain/brain_rev_2.sch (EAGLE design)
At the start: 15 parts, among them SW1 SPST_TACT-KMR2, U1 ATMEGA168, Y1 RESONATORSMD

Commit message: Furby
Parts:
- removed JP5: (no value), SparkFun_mod:M081X08
- added JP1: (no value), SparkFun:M081X08
Connections:
- net +5V: now also JP1.7; no longer JP5.7
- net A0: now also JP1.2; no longer JP5.2
- net A1: now also JP1.1; no longer JP5.1
- net A7: now also JP1.3; no longer JP5.3
- net D11: now also JP1.6; no longer JP5.6
- net D12: now also JP1.5; no longer JP5.5
- net D13: now also JP1.4; no longer JP5.4
- net V+: now also JP1.8; no longer JP5.8
Changed lines of the file:
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@@
 <part name="JP3" library="SparkFun_mod" deviceset="M02" device="PTH"/>
 <part name="P+1" library="supply1" deviceset="V+" device=""/>
-<part name="JP5" library="SparkFun_mod" deviceset="M08" device="1X08"/>
 <part name="U1" library="SparkFun" deviceset="ATMEGA168" device=""/>
 <part name="JP7" library="SparkFun" deviceset="ARDUINO_SERIAL_PROGRAM" device="PTH" value="FTDI Basic"/>
@@
 <part name="GND3" library="SparkFun" deviceset="GND" device=""/>
 <part name="SW1" library="adafruit" deviceset="SPST_TACT" device="-KMR2"/>
+<part name="JP1" library="SparkFun" deviceset="M08" device="1X08"/>
 </parts>
 <sheets>
@@
 <attribute name="VALUE" x="110.236" y="128.524" size="1.778" layer="96" rot="R90"/>
 </instance>
-<instance part="JP5" gate="G$1" x="132.08" y="30.48" rot="R180"/>
 <instance part="U1" gate="G$1" x="25.4" y="45.72"/>
 <instance part="JP7" gate="G$1" x="-58.42" y="50.8"/>
@@
 <instance part="GND3" gate="1" x="121.92" y="40.64" rot="R90"/>
 <instance part="SW1" gate="G$1" x="-20.32" y="78.74" rot="R270"/>
+<instance part="JP1" gate="G$1" x="132.08" y="30.48" rot="R180"/>
 </instances>
 <busses>
@@
 </segment>
 <segment>
-<pinref part="JP5" gate="G$1" pin="8"/>
 <pinref part="P+2" gate="1" pin="V+"/>
 <wire x1="127" y1="20.32" x2="121.92" y2="20.32" width="0.1524" layer="91"/>
+<pinref part="JP1" gate="G$1" pin="8"/>
+<junction x="127" y="20.32"/>
 </segment>
 </net>
@@
 <wire x1="50.8" y1="71.12" x2="91.44" y2="71.12" width="0.1524" layer="91"/>
 <wire x1="91.44" y1="71.12" x2="91.44" y2="35.56" width="0.1524" layer="91"/>
-<pinref part="JP5" gate="G$1" pin="2"/>
 <wire x1="91.44" y1="35.56" x2="127" y2="35.56" width="0.1524" layer="91"/>
+<pinref part="JP1" gate="G$1" pin="2"/>
+<junction x="127" y="35.56"/>
 </segment>
 </net>
@@
 </segment>
 <segment>
-<pinref part="JP5" gate="G$1" pin="7"/>
 <pinref part="P+3" gate="1" pin="+5V"/>
 <wire x1="127" y1="22.86" x2="121.92" y2="22.86" width="0.1524" layer="91"/>
+<pinref part="JP1" gate="G$1" pin="7"/>
+<junction x="127" y="22.86"/>
 </segment>
 </net>
@@
 <wire x1="93.98" y1="68.58" x2="93.98" y2="38.1" width="0.1524" layer="91"/>
 <wire x1="93.98" y1="38.1" x2="127" y2="38.1" width="0.1524" layer="91"/>
-<pinref part="JP5" gate="G$1" pin="1"/>
+<pinref part="JP1" gate="G$1" pin="1"/>
+<junction x="127" y="38.1"/>
 </segment>
 </net>
@@
 <wire x1="93.98" y1="17.78" x2="93.98" y2="25.4" width="0.1524" layer="91"/>
 <wire x1="93.98" y1="25.4" x2="127" y2="25.4" width="0.1524" layer="91"/>
-<pinref part="JP5" gate="G$1" pin="6"/>
+<pinref part="JP1" gate="G$1" pin="6"/>
+<junction x="127" y="25.4"/>
 </segment>
 </net>
@@
 <wire x1="50.8" y1="15.24" x2="91.44" y2="15.24" width="0.1524" layer="91"/>
 <wire x1="91.44" y1="15.24" x2="91.44" y2="27.94" width="0.1524" layer="91"/>
-<pinref part="JP5" gate="G$1" pin="5"/>
 <wire x1="91.44" y1="27.94" x2="127" y2="27.94" width="0.1524" layer="91"/>
+<pinref part="JP1" gate="G$1" pin="5"/>
+<junction x="127" y="27.94"/>
 </segment>
 </net>
@@
 <wire x1="50.8" y1="12.7" x2="88.9" y2="12.7" width="0.1524" layer="91"/>
 <wire x1="88.9" y1="12.7" x2="88.9" y2="30.48" width="0.1524" layer="91"/>
-<pinref part="JP5" gate="G$1" pin="4"/>
 <wire x1="88.9" y1="30.48" x2="127" y2="30.48" width="0.1524" layer="91"/>
+<pinref part="JP1" gate="G$1" pin="4"/>
+<junction x="127" y="30.48"/>
 </segment>
 </net>
@@
 <wire x1="50.8" y1="53.34" x2="88.9" y2="53.34" width="0.1524" layer="91"/>
 <wire x1="88.9" y1="53.34" x2="88.9" y2="33.02" width="0.1524" layer="91"/>
-<pinref part="JP5" gate="G$1" pin="3"/>
 <wire x1="88.9" y1="33.02" x2="127" y2="33.02" width="0.1524" layer="91"/>
-</segment>
-</net>
+<pinref part="JP1" gate="G$1" pin="3"/>
+<junction x="127" y="33.02"/>
+</segment>
+</net>
