File: osi/brain/brain_rev_3.brd (EAGLE design)
At the start: 25.4 x 25.4 mm, 13 parts, among them IC1 UA7805CKCS, IC2 MCP1702

Commit message: furby board production
Parts:
- removed C1: 0.33uF, adafruit:C025-024X044
- removed C2: 1uF, adafruit:C025-024X044
- removed D1: (no value), SparkFun:DIODE-1N4148
- removed F1: PTCPTH, SparkFun_mod:PTC
- removed IC1: UA7805CKCS, SparkFun:TO-220-ALT
- removed IC2: MCP1702, adafruit:TO92-INLINE
- removed LED1: (no value), adafruit:LED3MM
- removed R1: 1k, adafruit:0204/5
- removed U$1: 2.1MMJACKTHM, adafruit:PJ-102A
- removed U$2: (no value), DC_SYM:DC_POS_CTR
- removed U$3: (no value), DC_SYM:DC_POS_CTR-BOTTOM
- added JP1: (no value), SparkFun_mod:1X08
- added JP2: (no value), SparkFun:1X06
- moved JP6 25.4 mm to (27.9, 2.54)
- moved JP5 25.4 mm to (30.5, 22.9)
Connections:
- net D10 renamed A6
- removed net N$1: F1.P$1, U$1.TIP
- removed net N$2: LED1.K, R1.1
- new net N$12: JP2.3
- new net N$13: JP2.2
- new net N$14: JP2.1
- new net N$4: JP1.5
- new net N$5: JP1.4
- new net N$6: JP1.3
- new net N$7: JP1.2
- new net N$8: JP1.1
- net +3V3: now also JP2.4; no longer IC2.3
- net +5V: now also JP1.7; no longer C2.1, IC1.OUT, IC2.2, LED1.A
- net GND: now also JP2.5; no longer C1.2, C2.2, IC1.GND, IC2.1, R1.2, U$1.RING
- net N$3: now also JP1.6; no longer D1.A, F1.P$2
- net RESET: now also JP2.6
- net V+: now also JP1.8; no longer C1.1, D1.C, IC1.IN
Routing:
- net +5V: track 58.4 -> 0.00 mm
- net V+: track 53.1 -> 0.00 mm
- net +3V3: track 7.07 -> 0.00 mm
- net N$1: track 6.30 -> 0.00 mm
- net N$3: track 2.41 -> 0.00 mm
- net N$2: track 2.02 -> 0.00 mm
Other:
- board size 25.4 x 25.4 mm -> 50.8 x 25.4 mm
- board text added: "11"
- board text added: "12"
- board text added: "13"
- board text added: "A0"
- board text added: "A6"
- board text added: "A7"
- board text added: "Apr 12"
- board text added: "Atmega328"
- board text added: "NODE"
- board text added: "i2c"
- board text removed: "1.5A"
- board text removed: "1k"
- board text removed: "1uF"
- board text removed: "25V"
- board text removed: "3V: 0.25A"
- board text removed: "5V: 1.5A"
- board text removed: "7-25 VDC"
- board text removed: "Apr 13"
- board text removed: "D2"
- board text removed: "D3"
- board text removed: "D4"
- board text removed: "D5"
- board text removed: "D6"
- board text removed: "D7"
- board text removed: "MCP1702"
- board text removed: "PTC"
- board text removed: "PWR"
- board text removed: "UA7805CKCS"
