File: osi/batt/power-dc_rev_1.brd (EAGLE design)
At the start: 25.4 x 25.4 mm, 5 parts

Commit message: brain batt cleanup
Parts:
- removed I2C_L, I2C_R: (no value), SparkFun_mod:1X05
- removed RESET: PTS635_SWITCH, _my-parts:PTS635_SWITCH
- added BAT3: (no value), SparkFun_mod:BATTCOM_20MM_PTH
- added U$1: SWITCH, _my-parts:SWITCH
- JP6: value (none) -> 6
- JP8: value (none) -> 8
Connections:
- removed net RESET: RESET.P$2
- new net N$1: BAT3.2, U$1.3, U$1.6
- net +3V3: now also BAT3.1; no longer I2C_L.4, I2C_R.2
- net +5V: no longer I2C_L.5, I2C_R.1
- net GND: now also U$1.2, U$1.5; no longer I2C_L.3, I2C_R.3, RESET.P$1
- net SCL_D4: no longer I2C_L.1, I2C_R.5
- net SDA_D6: no longer I2C_L.2, I2C_R.4
Routing:
- net N$1: track 0.00 -> 24.7 mm
- net GND: track 0.00 -> 22.9 mm
- net +3V3: track 0.00 -> 19.6 mm
Other:
- board text added: "BATT"
- board text added: "Batt Rev 1 Feb 12"
- board text removed: "+5V"
- board text removed: "3V3"
- board text removed: "5V"
- board text removed: "Attiny 84"
- board text removed: "BRAIN"
- board text removed: "Brain Rev 1 Feb 12"
- board text removed: "D10"
- board text removed: "GND"
- board text removed: "RESET"
- board text removed: "SCK"
- board text removed: "SDA"
Changed lines of the file:
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@@
 <setting verticaltext="up"/>
 </settings>
-<grid distance="0.05" unitdist="inch" unit="inch" style="lines" multiple="1" display="yes" altdistance="0.005" altunitdist="inch" altunit="inch"/>
+<grid distance="0.025" unitdist="inch" unit="inch" style="lines" multiple="1" display="yes" altdistance="0.005" altunitdist="inch" altunit="inch"/>
 <layers>
 <layer number="1" name="Top" color="4" fill="1" visible="yes" active="yes"/>
@@
 <wire x1="0.000159375" y1="21.590159375" x2="0" y2="21.590159375" width="0" layer="20"/>
 <wire x1="0" y1="21.590159375" x2="0" y2="0" width="0" layer="20"/>
-<text x="25.146" y="0.381" size="0.8128" layer="21" font="vector" ratio="15" rot="R90">RESET</text>
 <text x="0.70358125" y="2.7432" size="0.8128" layer="21" font="vector" ratio="15">V+ GND 5V 3V3 D8 D9</text>
 <text x="4.480559375" y="21.72461875" size="0.9144" layer="21" font="vector" ratio="15">D7 D6 D5 D4 D3 D2 D1 D0</text>
-<text x="40.64" y="15.24" size="1.6764" layer="21" font="vector" ratio="10" rot="R90">Attiny 84</text>
-<text x="29.21" y="21.336" size="1.27" layer="21" font="vector" ratio="20">BRAIN</text>
+<text x="24.765" y="20.574" size="1.27" layer="21" font="vector" ratio="20" rot="R180">BATT</text>
 <text x="11.049" y="4.572" size="0.8128" layer="22" font="vector" ratio="15" rot="MR90">MakersBox.blogspot.com</text>
 <text x="13.462" y="4.318" size="1.27" layer="22" font="vector" ratio="15" rot="MR90">One Square Inch</text>
-<text x="37.084" y="18.415" size="0.8128" layer="22" font="vector" ratio="12" rot="MR270">Brain
+<text x="24.384" y="21.59" size="0.8128" layer="22" font="vector" ratio="12" rot="MR270">Batt
 Rev 1
 Feb 12</text>
-<text x="21.336" y="16.256" size="0.8128" layer="21" font="vector" ratio="10">3V3</text>
-<text x="21.336" y="13.589" size="0.8128" layer="21" font="vector" ratio="10">GND</text>
-<text x="21.336" y="11.049" size="0.8128" layer="21" font="vector" ratio="10">SDA</text>
-<text x="21.336" y="8.509" size="0.8128" layer="21" font="vector" ratio="10">SCK</text>
 <text x="23.530559375" y="21.72461875" size="0.9144" layer="22" font="vector" ratio="15" rot="MR0">D0 D1 D2 D3 D4 D5 D6 D7</text>
 <text x="14.67358125" y="2.7432" size="0.8128" layer="22" font="vector" ratio="15" rot="MR0">D8 D9 3V3 5V GND V+</text>
-<text x="20.955" y="17.399" size="0.6096" layer="22" font="vector" ratio="15" rot="MR270">3V3</text>
-<text x="20.955" y="14.859" size="0.6096" layer="22" font="vector" ratio="15" rot="MR270">GND</text>
-<text x="20.955" y="12.319" size="0.6096" layer="22" font="vector" ratio="15" rot="MR270">SDA</text>
-<text x="20.955" y="9.779" size="0.6096" layer="22" font="vector" ratio="15" rot="MR270">SCK</text>
-<text x="21.336" y="18.796" size="0.8128" layer="21" font="vector" ratio="10">+5V</text>
-<text x="30.099" y="12.954" size="0.6096" layer="21" font="vector" ratio="10" rot="R270">D10</text>
-<text x="20.955" y="19.685" size="0.6096" layer="22" font="vector" ratio="15" rot="MR270">5V</text>
 </plain>
 <attributes>
@@
 </autorouter>
 <elements>
-<element name="RESET" library="_my-parts" package="PTS635_SWITCH" value="PTS635_SWITCH" x="16.51" y="1.905"/>
-<element name="I2C_L" library="SparkFun_mod" package="1X05" value="" x="19.685" y="7.62" rot="R90"/>
-<element name="I2C_R" library="SparkFun_mod" package="1X05" value="" x="5.715" y="17.78" rot="R270"/>
-<element name="JP6" library="SparkFun" package="1X06" value="" x="1.27" y="1.27"/>
-<element name="JP8" library="SparkFun" package="1X08" value="" x="5.08" y="24.13"/>
+<element name="JP6" library="SparkFun" package="1X06" value="6" x="1.27" y="1.27"/>
+<element name="JP8" library="SparkFun" package="1X08" value="8" x="5.08" y="24.13"/>
+<element name="BAT3" library="SparkFun_mod" package="BATTCOM_20MM_PTH" value="" x="1.905" y="12.7"/>
+<element name="U$1" library="_my-parts" package="SWITCH" value="SWITCH" x="23.495" y="4.445" rot="R90"/>
 </elements>
 <signals>
@@
 <vertex x="-0.635" y="-0.635"/>
 </polygon>
-<contactref element="RESET" pad="P$1"/>
-<contactref element="I2C_L" pad="3"/>
-<contactref element="I2C_R" pad="3"/>
 <contactref element="JP6" pad="2"/>
-<wire x1="16.51" y1="1.905" x2="19.685" y2="12.7" width="0" layer="19" extent="1-1"/>
-<wire x1="5.715" y1="12.7" x2="19.685" y2="12.7" width="0" layer="19" extent="1-1"/>
-<wire x1="3.81" y1="1.27" x2="16.51" y2="1.905" width="0" layer="19" extent="1-1"/>
-</signal>
-<signal name="RESET">
-<contactref element="RESET" pad="P$2"/>
+<contactref element="U$1" pad="2"/>
+<contactref element="U$1" pad="5"/>
+<wire x1="24.257" y1="4.445" x2="20.955" y2="4.445" width="0.6096" layer="16"/>
+<wire x1="20.955" y1="4.445" x2="5.08" y2="4.445" width="0.6096" layer="16"/>
+<wire x1="5.08" y1="4.445" x2="3.81" y2="3.175" width="0.6096" layer="16"/>
+<wire x1="3.81" y1="3.175" x2="3.81" y2="1.27" width="0.6096" layer="16"/>
 </signal>
 <signal name="SDA_D6">
-<contactref element="I2C_L" pad="2"/>
-<contactref element="I2C_R" pad="4"/>
 <contactref element="JP8" pad="2"/>
-<wire x1="5.715" y1="10.16" x2="19.685" y2="10.16" width="0" layer="19" extent="1-1"/>
-<wire x1="7.62" y1="24.13" x2="5.715" y2="10.16" width="0" layer="19" extent="1-1"/>
 </signal>
 <signal name="SCL_D4">
-<contactref element="I2C_L" pad="1"/>
-<contactref element="I2C_R" pad="5"/>
 <contactref element="JP8" pad="4"/>
-<wire x1="5.715" y1="7.62" x2="19.685" y2="7.62" width="0" layer="19" extent="1-1"/>
-<wire x1="12.7" y1="24.13" x2="5.715" y2="7.62" width="0" layer="19" extent="1-1"/>
 </signal>
 <signal name="+3V3">
-<contactref element="I2C_L" pad="4"/>
-<contactref element="I2C_R" pad="2"/>
 <contactref element="JP6" pad="4"/>
-<wire x1="5.715" y1="15.24" x2="19.685" y2="15.24" width="0" layer="19" extent="1-1"/>
-<wire x1="8.89" y1="1.27" x2="5.715" y2="15.24" width="0" layer="19" extent="1-1"/>
+<contactref element="BAT3" pad="1"/>
+<wire x1="21.905" y1="12.7" x2="17.145" y2="12.7" width="0.6096" layer="1"/>
+<wire x1="17.145" y1="12.7" x2="8.89" y2="4.445" width="0.6096" layer="1"/>
+<wire x1="8.89" y1="4.445" x2="8.89" y2="1.27" width="0.6096" layer="1"/>
 </signal>
 <signal name="+5V">
-<contactref element="I2C_L" pad="5"/>
-<contactref element="I2C_R" pad="1"/>
 <contactref element="JP6" pad="3"/>
-<wire x1="5.715" y1="17.78" x2="19.685" y2="17.78" width="0" layer="19" extent="1-1"/>
-<wire x1="6.35" y1="1.27" x2="5.715" y2="17.78" width="0" layer="19" extent="1-1"/>
 </signal>
 <signal name="D8">
@@
 <contactref element="JP8" pad="1"/>
 </signal>
+<signal name="N$1">
+<contactref element="U$1" pad="6"/>
+<contactref element="BAT3" pad="2"/>
+<contactref element="U$1" pad="3"/>
+<wire x1="24.257" y1="6.985" x2="20.955" y2="6.985" width="0.6096" layer="16"/>
+<wire x1="20.955" y1="6.985" x2="7.62" y2="6.985" width="0.6096" layer="16"/>
+<wire x1="7.62" y1="6.985" x2="1.905" y2="12.7" width="0.6096" layer="16"/>
+</signal>
 </signals>
