File: osi/batt/power-dc_rev_1.sch (EAGLE design)
At the start: 8 parts, among them IC1 TINY24/44/84-PU

Commit message: brain batt cleanup
Parts:
- removed C1: (no value), SparkFun:CAPKIT
- removed IC1: TINY24/44/84-PU, avr-7:TINY24/44/84-PU
- removed JP1, JP2: (no value), SparkFun_mod:M05PTH
- removed JP3: (no value), SparkFun:M06SIP
- removed JP4: (no value), SparkFun:M081X08
- removed JP5: (no value), SparkFun_mod:M021X02_NO_SILK
- added BAT3: (no value), SparkFun_mod:BATTERY20PTH
- added JP6: 6, SparkFun:M06SIP
- added JP8: 8, SparkFun:M081X08
- U$1: value PTS635_SWITCH -> SWITCH; device _my-parts:PTS635_SWITCH -> _my-parts:SWITCH
Connections:
- removed net D10: IC1.(PCINT8/XTAL1/CLKI)PB0, JP5.1
- removed net RESET: IC1.(PCINT11/RESET/DW)PB3, U$1.P$2
- new net N$1: BAT3.-, U$1.3, U$1.6
- net +3V3: now also BAT3.+, JP6.4; no longer C1.2, IC1.VCC, JP1.4, JP2.2, JP3.4
- net +5V: now also JP6.3; no longer JP1.5, JP2.1, JP3.3
- net AREF_D0: now also JP8.8; no longer IC1.(PCINT0/AREF/ADC0)PA0, JP4.8
- net D1: now also JP8.7; no longer IC1.(PCINT1/AIN0/ADC1)PA1, JP4.7
- net D2: now also JP8.6; no longer IC1.(PCINT2/AIN1/ADC2)PA2, JP4.6
- net D3: now also JP8.5; no longer IC1.(PCINT3/T0/ADC3)PA3, JP4.5
- net D5: now also JP8.3; no longer IC1.(PCINT5/OC1B/MISO/DO/ADC5)PA5, JP4.3
- net D7: now also JP8.1; no longer IC1.(PCINT7/ICP/OC0B/ADC7)PA7, JP4.1
- net D8: now also JP6.5; no longer IC1.(PCINT10/INT0/OC0A/CKOUT)PB2, JP3.5
- net D9: now also JP6.6; no longer IC1.(PCINT9/XTAL2)PB1, JP3.6
- net GND: now also JP6.2, U$1.2, U$1.5; no longer C1.1, IC1.GND, JP1.3, JP2.3, JP3.2, JP5.2, U$1.P$1
- net SCL_D4: now also JP8.4; no longer IC1.(PCINT4/T1/SCL/USCK/ADC4)PA4, JP1.1, JP2.5, JP4.4
- net SDA_D6: now also JP8.2; no longer IC1.(PCINT6/OC1A/SDA/MOSI/ADC6)PA6, JP1.2, JP2.4, JP4.2
- net V+: now also JP6.1; no longer JP3.1
