File: osi/power/power-ac_rev_1.sch (EAGLE design)
At the start: 8 parts, among them IC1 TINY24/44/84-PU

Commit message: control brain
Parts:
- removed IC2_L, IC2_R: (no value), SparkFun_mod:M05PTH
- removed JP8: (no value), SparkFun:M081X08
- added C6: (no value), SparkFun:CAP_POLPTH1
- added D1: (no value), SparkFun:DIODE1N4148
- added F1: PTCPTH, SparkFun_mod:PTCPTH
- added IC2: (no value), adafruit:MCP1700INLINE
- added JP5: (no value), SparkFun:M06SIP
- added LED1: (no value), adafruit:LED3MM
- C1: device SparkFun:CAPKIT -> SparkFun:CAP_POLPTH1
- IC1: value TINY24/44/84-PU -> (none); device avr-7:TINY24/44/84-PU -> SparkFun:V_REG_78XX-TO-220
- JP6: device SparkFun:M06SIP -> SparkFun:M081X08
- R1: device adafruit_mod:R-US_0204/2V -> adafruit:R-US_0204/2V
- U$1: value PTS635_SWITCH -> 2.1MMJACKTHM; device _my-parts:PTS635_SWITCH -> adafruit:2.1MMJACKTHM
Connections:
- removed net D10: IC1.(PCINT8/XTAL1/CLKI)PB0, JP6.6
- removed net RESET: IC1.(PCINT11/RESET/DW)PB3, U$1.P$2
- new net N$1: F1.1, U$1.TIP
- new net N$2: LED1.C, R1.2
- new net N$3: D1.A, F1.2
- net +3V3: now also IC2.OUT, JP5.4; no longer C1.2, IC1.VCC, IC2_L.4, IC2_R.2, JP6.4
- net +5V: now also C1.+, IC1.OUT, IC2.IN, JP5.3, LED1.A; no longer IC2_L.5, IC2_R.1, JP6.3
- net AREF_D0: now also JP6.8; no longer IC1.(PCINT0/AREF/ADC0)PA0, JP8.8
- net D1: now also JP6.7; no longer IC1.(PCINT1/AIN0/ADC1)PA1, JP8.7
- net D2: now also JP6.6; no longer IC1.(PCINT2/AIN1/ADC2)PA2, JP8.6
- net D3: now also JP6.5; no longer IC1.(PCINT3/T0/ADC3)PA3, JP8.5
- net D5: now also JP6.3; no longer IC1.(PCINT5/OC1B/MISO/DO/ADC5)PA5, JP8.3
- net D7: now also JP6.1; no longer IC1.(PCINT7/ICP/OC0B/ADC7)PA7, JP8.1
- net D8: now also JP5.5; no longer IC1.(PCINT10/INT0/OC0A/CKOUT)PB2, R1.1
- net D9: now also JP5.6; no longer IC1.(PCINT9/XTAL2)PB1, JP6.5
- net GND: now also C1.-, C6.-, IC2.GND, JP5.2, R1.1, U$1.RING; no longer C1.1, IC2_L.3, IC2_R.3, JP6.2, R1.2, U$1.P$1
- net SCL_D4: now also JP6.4; no longer IC1.(PCINT4/T1/SCL/USCK/ADC4)PA4, IC2_L.1, IC2_R.5, JP8.4
- net SDA_D6: now also JP6.2; no longer IC1.(PCINT6/OC1A/SDA/MOSI/ADC6)PA6, IC2_L.2, IC2_R.4, JP8.2
- net V+: now also C6.+, D1.C, IC1.IN, JP5.1; no longer JP6.1
Other:
- moved on the sheet: R1
