File: osi/power/power_rev_2.brd (EAGLE design)
At the start: 25.4 x 25.4 mm, 13 parts, among them IC1 UA7805CKCS, IC2 MCP1702

Commit message: moving headers
Parts:
- removed JP5: (no value), SparkFun_mod:1X08
- added JP1: (no value), SparkFun:1X08
- moved JP6 1.27 mm to (2.54, 1.27)
Connections:
- net +5V: now also JP1.7; no longer JP5.7
- net A0: now also JP1.2; no longer JP5.2
- net A1: now also JP1.1; no longer JP5.1
- net A7: now also JP1.3; no longer JP5.3
- net D11: now also JP1.6; no longer JP5.6
- net D12: now also JP1.5; no longer JP5.5
- net D13: now also JP1.4; no longer JP5.4
- net V+: now also JP1.8; no longer JP5.8
Routing:
- net V+: track 53.1 -> 34.5 mm
- net +5V: track 58.4 -> 56.9 mm
- net +3V3: track 7.07 -> 8.06 mm
Other:
- board text removed: "UA7805CKCS"
