File: osi/control/control_rev_1.brd (EAGLE design)
At the start: 25.4 x 25.4 mm, 13 parts, among them J1 1X2-3.5MM, J2 1X2-3.5MM

Commit message: rev 1 manufacture
Changed lines of the file:
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@@
 <setting verticaltext="up"/>
 </settings>
-<grid distance="0.01" unitdist="inch" unit="inch" style="lines" multiple="1" display="yes" altdistance="0.005" altunitdist="inch" altunit="inch"/>
+<grid distance="0.05" unitdist="inch" unit="inch" style="lines" multiple="1" display="yes" altdistance="0.005" altunitdist="inch" altunit="inch"/>
 <layers>
 <layer number="1" name="Top" color="4" fill="1" visible="yes" active="yes"/>
@@
 <text x="4.318" y="15.748" size="1.778" layer="22" font="vector" ratio="15" rot="MR0">A</text>
 <text x="22.606" y="15.494" size="1.778" layer="22" font="vector" ratio="15" rot="MR0">B</text>
-<text x="21.082" y="15.24" size="1.778" layer="21" font="vector" ratio="15">B</text>
-<text x="3.302" y="15.24" size="1.778" layer="21" font="vector" ratio="15">A</text>
+<text x="21.463" y="15.494" size="1.778" layer="21" font="vector" ratio="15">B</text>
+<text x="3.048" y="15.875" size="1.778" layer="21" font="vector" ratio="15">A</text>
 <text x="0.635" y="10.922" size="1.016" layer="21" font="vector" ratio="15" rot="SR270">V+</text>
 <text x="0.635" y="8.382" size="1.016" layer="21" font="vector" ratio="15" rot="SR270">5V</text>
