File: osi/control/control_rev_2.sch (EAGLE design)
At the start: 15 parts, among them U1 ATMEGA168, Y1 RESONATORSMD

Commit message: 328p surface mount
Parts:
- removed C1, C2: (no value), SparkFun:CAP1206
- removed LED1: (no value), adafruit:LEDCHIPLED_1206
- removed R1, R2, R3, R4: (no value), SparkFun:RESISTOR1206
- removed S1: (no value), SparkFun:TAC_SWITCHSMD
- removed U1: ATMEGA168, SparkFun:ATMEGA168
- removed Y1: RESONATORSMD, SparkFun:RESONATORSMD
Connections:
- removed net A0: JP5.2, U1.PC0(ADC0)
- removed net A1: JP5.1, U1.PC1(ADC1)
- removed net A6: U1.ADC6
- removed net D2: U1.PD2(INT0)
- removed net D3: LED1.A, U1.PD3(INT1)
- removed net D4: U1.PD4(XCK/T0)
- removed net D5: U1.PD5(T1)
- removed net D6: U1.PD6(AIN0)
- removed net D7: U1.PD7(AIN1)
- removed net D8: U1.PB0(ICP)
- removed net D9: U1.PB1(OC1A)
- removed net N$1: U1.PB7(XTAL2/TOSC2), Y1.3
- removed net N$3: U1.PB6(XTAL1/TOSC1), Y1.1
- removed net N$4: LED1.C, R1.1
- net +3V3: no longer C2.1, R2.1, R3.2, R4.2, U1.AREF, U1.AVCC, U1.VCC@1, U1.VCC@2
- net A2: no longer U1.PC2(ADC2)
- net A3: no longer U1.PC3(ADC3)
- net A7: no longer U1.ADC7
- net D10: no longer U1.PB2(SS/OC1B)
- net D11: no longer U1.PB3(MOSI/OC2)
- net D12: no longer U1.PB4(MISO)
- net D13: no longer U1.PB5(SCK)
- net DTR: no longer C1.1
- net GND: no longer C2.2, R1.2, S1.2, U1.AGND, U1.GND@1, U1.GND@2, Y1.2
- net RESET: no longer C1.2, R2.2, S1.3, U1.PC6(/RESET)
- net RXI: no longer U1.PD0(RXD)
- net SCL_A5: no longer R3.1, U1.PC5(ADC5/SCL)
- net SDA_A4: no longer R4.1, U1.PC4(ADC4/SDA)
- net TXO: no longer U1.PD1(TXD)

Commit message: layout changes
Parts:
- removed JP2: (no value), SparkFun_mod:M04PTH
- removed JP3: (no value), SparkFun_mod:M02PTH
- removed JP7: FTDI Basic, SparkFun:ARDUINO_SERIAL_PROGRAMPTH
- added C1, C2: 100uF/16V, rcl-ez:CPOL-USE2.5-6
- added C3: 0.1uF, rcl-ez:C-US025-025X050
- added JP1: (no value), adafruit_mod:PINHD-1X3
- added MTR1, MTR2: TERMINAL, _my-parts:TERMINAL
- added TRACKS: L293D, texas:L293E
Connections:
- net D10 renamed A6
- removed net DTR: JP7.DTR
- removed net RXI: JP7.TXO
- removed net SCL_A5: JP2.1
- removed net SDA_A4: JP2.2
- removed net TXO: JP7.RXI
- new net A0: JP5.2, TRACKS.3A
- new net A1: JP5.1, TRACKS.4A
- new net N$1: MTR1.P$1, TRACKS.1Y
- new net N$2: MTR2.P$1, TRACKS.4Y
- new net N$3: MTR1.P$3, TRACKS.2Y
- new net N$4: MTR2.P$3, TRACKS.3Y
- new net N$8: C2.+, JP1.2, TRACKS.VCC2
- net +3V3: no longer JP2.4, JP7.VCC
- net +5V: now also C1.+, C3.1, JP1.1, TRACKS.VCC1; no longer JP3.2
- net A2: now also TRACKS.1A
- net A3: now also TRACKS.2A
- net D12: now also TRACKS.1-2EN
- net D13: now also TRACKS.3-4EN
- net GND: now also C1.-, C2.-, C3.2, MTR1.P$2, MTR2.P$2, TRACKS.GND1, TRACKS.GND2, TRACKS.GND3, TRACKS.GND4; no longer JP2.3, JP7.CTS, JP7.GND
- net V+: now also JP1.3; no longer JP3.1

Commit message: FURBY
Changed lines of the file:
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@@
 <wire x1="40.64" y1="58.42" x2="12.7" y2="58.42" width="0.1524" layer="91"/>
 <wire x1="40.64" y1="71.12" x2="40.64" y2="58.42" width="0.1524" layer="91"/>
+<label x="15.24" y="58.42" size="1.778" layer="95"/>
 </segment>
 </net>
@@
 <wire x1="43.18" y1="83.82" x2="12.7" y2="83.82" width="0.1524" layer="91"/>
 <wire x1="43.18" y1="68.58" x2="43.18" y2="83.82" width="0.1524" layer="91"/>
+<label x="15.24" y="83.82" size="1.778" layer="95"/>
 </segment>
 </net>
@@
 <wire x1="53.34" y1="53.34" x2="53.34" y2="12.7" width="0.1524" layer="91"/>
 <wire x1="53.34" y1="12.7" x2="60.96" y2="12.7" width="0.1524" layer="91"/>
+<label x="15.24" y="53.34" size="1.778" layer="95"/>
 </segment>
 </net>
@@
 <label x="121.92" y="86.36" size="1.778" layer="95"/>
 <wire x1="45.72" y1="63.5" x2="109.22" y2="63.5" width="0.1524" layer="91"/>
+<label x="-20.32" y="58.42" size="1.778" layer="95"/>
 </segment>
 </net>
@@
 <label x="121.92" y="88.9" size="1.778" layer="95"/>
 <wire x1="48.26" y1="66.04" x2="106.68" y2="66.04" width="0.1524" layer="91"/>
+<label x="-20.32" y="83.82" size="1.778" layer="95"/>
 </segment>
 </net>
@@
 <label x="88.646" y="17.272" size="1.778" layer="95" rot="R180"/>
 <label x="121.92" y="27.94" size="1.778" layer="95"/>
-</segment>
-</net>
+<label x="-22.86" y="91.44" size="1.778" layer="95"/>
+</segment>
+</net>
