File: osi/isp/isp_02.brd (EAGLE design)
At the start: 25.4 x 25.4 mm, 8 parts

Commit message: 328 TFOP?
Parts:
- removed I2C_L, I2C_R: (no value), SparkFun_mod:1X05
- removed JP8: (no value), SparkFun:1X08
- removed R1, R2: (no value), adafruit_mod:0204V
- removed RESET: PTS635_SWITCH, _my-parts:PTS635_SWITCH
- added ISP1: AVRISP-6, adafruit:AVRISP
- added JP5: (no value), SparkFun_mod:1X08
- U$1: value AVR-MEGA8-AI -> PTS635_SWITCH; device SparkFun:TQFP32-08 -> _my-parts:PTS635_SWITCH
- moved U$1 16.0 mm to (23.1, 1.78), turned to 180 degrees
Connections:
- removed net AREF_D0: JP8.8
- removed net D1: JP8.7, R2.2
- removed net D10: JP6.6
- removed net D2: JP8.6, R1.2
- removed net D3: JP8.5
- removed net D5: JP8.3
- removed net D7: JP8.1
- removed net D8: JP6.5
- removed net SCL_D4: I2C_L.1, I2C_R.5, JP8.4
- removed net SDA_D6: I2C_L.2, I2C_R.4, JP8.2
- new net D11: ISP1.4, JP5.7
- new net D12: ISP1.1, JP5.6
- new net D13: ISP1.3, JP5.5
- net +3V3: now also ISP1.2; no longer I2C_L.4, I2C_R.2
- net +5V: no longer I2C_L.5, I2C_R.1
- net GND: now also ISP1.6, U$1.P$1; no longer I2C_L.3, I2C_R.3, R1.1, R2.1, RESET.P$1
- net RESET: now also ISP1.5, JP6.6, U$1.P$2; no longer RESET.P$2
Routing:
- net D13: track 0.00 -> 21.9 mm
- net D12: track 0.00 -> 18.2 mm
- net +3V3: track 0.00 -> 15.0 mm
- net D11: track 0.00 -> 13.8 mm
- net RESET: track 0.00 -> 13.1 mm
Other:
- outline, holes or cut-outs redrawn
- board text added: "A0"
- board text added: "A1"
- board text added: "A2"
- board text added: "A3"
- board text added: "A4"
- board text added: "Apr 12"
- board text added: "D11"
- board text added: "D12"
- board text added: "D13"
- board text added: "ISP"
- board text added: "MISO"
- board text added: "MOSI"
- board text added: "RST"
- board text removed: "+5V"
- board text removed: "BRAIN"
- board text removed: "Brain Rev 1 Feb 12"
- board text removed: "D0"
- board text removed: "D1"
- board text removed: "D2"
- board text removed: "D3"
- board text removed: "D4"
- board text removed: "D5"
- board text removed: "D6"
- board text removed: "D7"
- board text removed: "One Square Inch"
- board text removed: "SDA"
