File: osi/isp/isp_2.brd (EAGLE design)
At the start: 25.4 x 25.4 mm, 9 parts

Commit message: layout changes
Parts:
- removed C1, C2: 100uF/16V, rcl-ez:E2,5-6
- removed C3: 0.1uF, rcl-ez:C025-025X050
- removed JP1: (no value), adafruit_mod:1X03
- removed MTR1, MTR2: TERMINAL, _my-parts:TERMINAL_3
- removed TRACKS: L293D, texas:DIL16
- added J1: AVR_SPI_PRG_6PTH, SparkFun:2X3
Connections:
- net A6 renamed D10
- removed net N$1: MTR1.P$1, TRACKS.3
- removed net N$2: MTR2.P$1, TRACKS.14
- removed net N$3: MTR1.P$3, TRACKS.6
- removed net N$4: MTR2.P$3, TRACKS.11
- removed net N$8: C2.+, JP1.2, TRACKS.8
- net +3V3: now also J1.2
- net +5V: no longer C1.+, C3.1, JP1.1, TRACKS.16
- net A0: no longer TRACKS.10
- net A1: no longer TRACKS.15
- net A2: no longer TRACKS.2
- net A3: no longer TRACKS.7
- net D11: now also J1.4
- net D12: now also J1.1; no longer TRACKS.1
- net D13: now also J1.3; no longer TRACKS.9
- net GND: now also J1.6; no longer C1.-, C2.-, C3.2, MTR1.P$2, MTR2.P$2, TRACKS.12, TRACKS.13, TRACKS.4, TRACKS.5
- net RESET: now also J1.5
- net V+: no longer JP1.3
Routing:
- net +5V: track 51.3 -> 0.00 mm
- net A3: track 33.9 -> 0.00 mm
- net A0: track 22.9 -> 0.00 mm
- net D12: track 32.0 -> 9.20 mm
- net +3V3: track 0.00 -> 21.9 mm
- net N$3: track 14.9 -> 0.00 mm
- net N$8: track 13.6 -> 0.00 mm
- net N$1: track 13.1 -> 0.00 mm
- net V+: track 11.5 -> 0.00 mm
- net A1: track 10.9 -> 0.00 mm
- net RESET: track 0.00 -> 9.20 mm
- net N$2: track 8.30 -> 0.00 mm
- net D13: track 18.9 -> 12.8 mm
- net N$4: track 5.76 -> 0.00 mm
- net D11: track 7.67 -> 12.5 mm
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Other:
- board text added: "10"
- board text added: "D10"
- board text added: "ISP"
- board text added: "MISO"
- board text added: "MOSI"
- board text added: "PWR"
- board text added: "SCK"
- board text removed: "100uf"
- board text removed: "<-sel->"
- board text removed: "A6"
- board text removed: "CNTRL"
- board text removed: "CTRL"
- board text removed: "LM293"
