File: osi/isp/isp_rev_3.brd (EAGLE design)
At the start: 24.8 x 25.4 mm, 4 parts

Commit message: double board finished?
Parts:
- removed JP2: (no value), SparkFun_mod:1X06
- added J1: AVR_SPI_PRG_6PTH, SparkFun:2X3
- added U$1: NUNCHUCKCHUCK, _my-parts:CONN
- added U$2: (no value), _my-parts:OREGON_18_52
- moved JP6 30.2 mm to (22.2, 24.1), turned to 180 degrees
- moved JP5 27.1 mm to (19.7, 1.27), turned to 180 degrees
- moved JP1 12.1 mm to (1.91, 3.81), turned to 0 degrees
Connections:
- removed net RXI: JP1.2, JP2.3
- removed net TXO: JP1.1, JP2.2
- new net SCL_A5: JP1.2, U$1.SCL
- new net SDA_A4: JP1.1, U$1.SDA
- net +3V3: now also J1.2; no longer JP2.4
- net D3_D11: now also J1.4
- net D4_D12: now also J1.1
- net D7_D13: now also J1.3
- net DTR: no longer JP2.1
- net GND: now also J1.6; no longer JP2.5, JP2.6
- net RESET: now also J1.5
Routing:
- net D7_D13: track 0.00 -> 24.0 mm
- net RESET: track 0.00 -> 22.5 mm
- net D4_D12: track 0.00 -> 19.8 mm
- net SDA_A4: track 0.00 -> 16.1 mm, vias 0 -> 1
- net D3_D11: track 0.00 -> 15.1 mm
- net SCL_A5: track 0.00 -> 12.5 mm
- net +3V3: track 0.00 -> 11.6 mm
Other:
- outline, holes or cut-outs redrawn
- board text added: "I2C"
- board text added: "I2C / ISP"
- board text added: "ISP"
- board text added: "MISO"
- board text added: "MOSI"
- board text added: "May 13"
- board text added: "SCK"
- board text added: "SCL"
- board text added: "SDA"
- board text added: "VCC"
- board text removed: "3V3"
- board text removed: "5V"
- board text removed: "Apr 12"
- board text removed: "NODE"
- board text removed: "RXi"
- board text removed: "TXo"
- board text removed: "V+"
