File: osi/isp/isp_rev_3.sch (EAGLE design)
At the start: 4 parts

Commit message: double board finished?
Parts:
- removed JP2: (no value), SparkFun_mod:M06SIP
- added J1: AVR_SPI_PRG_6PTH, SparkFun:AVR_SPI_PRG_6PTH
- added U$1: NUNCHUCKCHUCK, _my-parts:NUNCHUCKCHUCK
Connections:
- removed net RXI: JP1.2, JP2.3
- removed net TXO: JP1.1, JP2.2
- new net SCL_A5: JP1.2, U$1.SCL
- new net SDA_A4: JP1.1, U$1.SDA
- net +3V3: now also J1.2; no longer JP2.4
- net D3_D11: now also J1.4
- net D4_D12: now also J1.1
- net D7_D13: now also J1.3
- net DTR: no longer JP2.1
- net GND: now also J1.6; no longer JP2.5, JP2.6
- net RESET: now also J1.5
Other:
- moved on the sheet: JP1
Changed lines of the file:
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@@
 <part name="JP5" library="SparkFun_mod" deviceset="M08" device="1X08"/>
 <part name="GND" library="_my-parts" deviceset="ADDRESSING" device="" value="GND"/>
-<part name="JP2" library="SparkFun_mod" deviceset="M06" device="SIP"/>
 <part name="JP1" library="SparkFun_mod" deviceset="M02" device="PTH"/>
+<part name="U$1" library="_my-parts" deviceset="NUNCHUCK" device="CHUCK"/>
+<part name="J1" library="SparkFun" deviceset="AVR_SPI_PRG_6" device="PTH"/>
+<part name="GND1" library="SparkFun" deviceset="GND" device=""/>
+<part name="+3V1" library="supply1" deviceset="+3V3" device=""/>
 </parts>
 <sheets>
@@
 <instance part="JP5" gate="G$1" x="132.08" y="30.48" rot="R180"/>
 <instance part="GND" gate="G$1" x="124.46" y="53.34"/>
-<instance part="JP2" gate="G$1" x="-27.94" y="27.94"/>
-<instance part="JP1" gate="G$1" x="73.66" y="45.72"/>
+<instance part="JP1" gate="G$1" x="76.2" y="76.2" rot="R180"/>
+<instance part="U$1" gate="G$1" x="55.88" y="83.82" rot="R180"/>
+<instance part="J1" gate="G$1" x="91.44" y="27.94" rot="R180"/>
+<instance part="GND1" gate="1" x="78.74" y="30.48" smashed="yes" rot="R270">
+<attribute name="VALUE" x="73.406" y="29.464" size="1.778" layer="96"/>
+</instance>
+<instance part="+3V1" gate="G$1" x="78.74" y="25.4" smashed="yes" rot="R90">
+<attribute name="VALUE" x="78.486" y="26.416" size="1.778" layer="96" rot="R180"/>
+</instance>
 </instances>
 <busses>
@@
 </segment>
 <segment>
-<wire x1="-22.86" y1="33.02" x2="-10.16" y2="33.02" width="0.1524" layer="91"/>
-<label x="-15.24" y="33.02" size="1.778" layer="95"/>
-<pinref part="JP2" gate="G$1" pin="5"/>
-<junction x="-22.86" y="33.02"/>
-</segment>
-<segment>
-<wire x1="-22.86" y1="35.56" x2="-10.16" y2="35.56" width="0.1524" layer="91"/>
-<label x="-15.24" y="35.56" size="1.778" layer="95"/>
-<pinref part="JP2" gate="G$1" pin="6"/>
-<junction x="-22.86" y="35.56"/>
+<pinref part="J1" gate="G$1" pin="6"/>
+<pinref part="GND1" gate="1" pin="GND"/>
 </segment>
 </net>
 <net name="RESET" class="0">
 <segment>
-<wire x1="127" y1="76.2" x2="119.38" y2="76.2" width="0.1524" layer="91"/>
 <pinref part="JP6" gate="G$1" pin="6"/>
 <label x="119.38" y="76.2" size="1.778" layer="95"/>
+<wire x1="127" y1="76.2" x2="109.22" y2="76.2" width="0.1524" layer="91"/>
+<wire x1="109.22" y1="76.2" x2="109.22" y2="30.48" width="0.1524" layer="91"/>
+<pinref part="J1" gate="G$1" pin="5"/>
+<wire x1="109.22" y1="30.48" x2="99.06" y2="30.48" width="0.1524" layer="91"/>
 </segment>
 </net>
@@
 </segment>
 <segment>
-<wire x1="-22.86" y1="30.48" x2="-10.16" y2="30.48" width="0.1524" layer="91"/>
-<label x="-15.24" y="30.48" size="1.778" layer="95"/>
-<pinref part="JP2" gate="G$1" pin="4"/>
-<junction x="-22.86" y="30.48"/>
+<pinref part="J1" gate="G$1" pin="2"/>
+<pinref part="+3V1" gate="G$1" pin="+3V3"/>
 </segment>
 </net>
@@
 <segment>
 <pinref part="JP6" gate="G$1" pin="2"/>
-<wire x1="111.76" y1="86.36" x2="127" y2="86.36" width="0.1524" layer="91"/>
+<wire x1="106.68" y1="86.36" x2="127" y2="86.36" width="0.1524" layer="91"/>
 <label x="116.84" y="86.36" size="1.778" layer="95"/>
+<wire x1="106.68" y1="86.36" x2="106.68" y2="25.4" width="0.1524" layer="91"/>
+<pinref part="J1" gate="G$1" pin="1"/>
+<wire x1="99.06" y1="25.4" x2="106.68" y2="25.4" width="0.1524" layer="91"/>
 </segment>
 </net>
@@
 <net name="SDA_A4" class="0">
 <segment>
-<label x="94.615" y="62.865" size="1.778" layer="95" rot="R180"/>
-<wire x1="93.98" y1="60.96" x2="81.28" y2="60.96" width="0.1524" layer="91"/>
+<label x="66.675" y="78.105" size="1.778" layer="95" rot="R180"/>
+<wire x1="68.58" y1="76.2" x2="53.34" y2="76.2" width="0.1524" layer="91"/>
+<pinref part="U$1" gate="G$1" pin="SDA"/>
+<pinref part="JP1" gate="G$1" pin="1"/>
 </segment>
 </net>
 <net name="SCL_A5" class="0">
 <segment>
-<label x="94.615" y="60.325" size="1.778" layer="95" rot="R180"/>
-<wire x1="93.98" y1="58.42" x2="81.28" y2="58.42" width="0.1524" layer="91"/>
+<label x="66.675" y="75.565" size="1.778" layer="95" rot="R180"/>
+<wire x1="68.58" y1="73.66" x2="53.34" y2="73.66" width="0.1524" layer="91"/>
+<pinref part="U$1" gate="G$1" pin="SCL"/>
+<pinref part="JP1" gate="G$1" pin="2"/>
 </segment>
 </net>
@@
 </segment>
 </net>
-<net name="TXO" class="0">
-<segment>
-<wire x1="81.28" y1="45.72" x2="86.36" y2="45.72" width="0.1524" layer="91"/>
-<label x="83.82" y="45.72" size="1.778" layer="95"/>
-<pinref part="JP1" gate="G$1" pin="1"/>
-</segment>
-<segment>
-<wire x1="-22.86" y1="25.4" x2="-10.16" y2="25.4" width="0.1524" layer="91"/>
-<label x="-15.24" y="25.4" size="1.778" layer="95"/>
-<pinref part="JP2" gate="G$1" pin="2"/>
-<junction x="-22.86" y="25.4"/>
-</segment>
-</net>
-<net name="RXI" class="0">
-<segment>
-<wire x1="81.28" y1="48.26" x2="86.36" y2="48.26" width="0.1524" layer="91"/>
-<label x="83.82" y="48.26" size="1.778" layer="95"/>
-<pinref part="JP1" gate="G$1" pin="2"/>
-</segment>
-<segment>
-<wire x1="-22.86" y1="27.94" x2="-10.16" y2="27.94" width="0.1524" layer="91"/>
-<label x="-15.24" y="27.94" size="1.778" layer="95"/>
-<pinref part="JP2" gate="G$1" pin="3"/>
-<junction x="-22.86" y="27.94"/>
-</segment>
-</net>
 <net name="D3_D11" class="0">
 <segment>
 <pinref part="JP5" gate="G$1" pin="3"/>
-<wire x1="114.3" y1="33.02" x2="127" y2="33.02" width="0.1524" layer="91"/>
 <label x="116.84" y="33.02" size="1.778" layer="95"/>
+<wire x1="127" y1="33.02" x2="101.6" y2="33.02" width="0.1524" layer="91"/>
+<wire x1="101.6" y1="33.02" x2="101.6" y2="38.1" width="0.1524" layer="91"/>
+<pinref part="J1" gate="G$1" pin="4"/>
+<wire x1="81.28" y1="27.94" x2="68.58" y2="27.94" width="0.1524" layer="91"/>
+<wire x1="101.6" y1="38.1" x2="68.58" y2="38.1" width="0.1524" layer="91"/>
+<wire x1="68.58" y1="38.1" x2="68.58" y2="27.94" width="0.1524" layer="91"/>
 </segment>
 </net>
@@
 <wire x1="111.76" y1="83.82" x2="127" y2="83.82" width="0.1524" layer="91"/>
 <label x="116.84" y="83.82" size="1.778" layer="95"/>
+<wire x1="111.76" y1="83.82" x2="111.76" y2="27.94" width="0.1524" layer="91"/>
+<pinref part="J1" gate="G$1" pin="3"/>
+<wire x1="99.06" y1="27.94" x2="101.6" y2="27.94" width="0.1524" layer="91"/>
+<wire x1="101.6" y1="27.94" x2="104.14" y2="27.94" width="0.1524" layer="91"/>
+<wire x1="111.76" y1="27.94" x2="104.14" y2="27.94" width="0.1524" layer="91"/>
 </segment>
 </net>
 <net name="DTR" class="0">
 <segment>
-<wire x1="-22.86" y1="22.86" x2="-10.16" y2="22.86" width="0.1524" layer="91"/>
-<label x="-15.24" y="22.86" size="1.778" layer="95"/>
-<pinref part="JP2" gate="G$1" pin="1"/>
-<junction x="-22.86" y="22.86"/>
-</segment>
-<segment>
 <pinref part="JP5" gate="G$1" pin="6"/>
