File: osi/chuck/chuck_rev_2.sch (EAGLE design)
At the start: 2 parts

Commit message: layout changes
Parts:
- added CHUCK: NUNCHUCK, _my-parts:NUNCHUCK
- added J1: AVR_SPI_PRG_6NS, SparkFun:AVR_SPI_PRG_6NS
- added JP2: (no value), SparkFun_mod:M04PTH
- added JP3: (no value), SparkFun_mod:M02PTH
Connections:
- net A6 renamed D10
- new net SCL_A5: CHUCK.SCL, JP2.1
- new net SDA_A4: CHUCK.SDA, JP2.2
- net +3V3: now also CHUCK.PWR, J1.2, JP2.4
- net +5V: now also JP3.2
- net D11: now also J1.4
- net D12: now also J1.1
- net D13: now also J1.3
- net GND: now also CHUCK.GND, J1.6, JP2.3
- net RESET: now also J1.5
- net V+: now also JP3.1
