File: furby/furby.sch (EAGLE design)
At the start: 38 parts, among them IC1 ATMEGA168PROUND, J1 1X2-3.5MM

Commit message: FURBY
Parts:
- removed 328, LEFT: M14, SparkFun:M14
- added C5: (no value), adafruit:C-US050-025X075
- added D1: (no value), adafruit:DIODEDO-1N4148
- added IC2: 74AC14N, 74xx-eu:74AC14N
- added JP1, JP2: M14, SparkFun_mod:M14
- added JP3: (no value), SparkFun:M02PTH
- added R10: 11.9k, adafruit:R-US_0204/7
- added R11: 15.7k, adafruit:R-US_0204/7
Connections:
- new net N$3: D1.A, JP3.2, R10.2, R11.1
- new net N$4: C5.1, D1.C, IC2A.I, JP3.1, R11.2
- new net N$8: IC2A.O
- net A0: now also JP1.9; no longer 328.9
- net A1: now also JP1.10; no longer 328.10
- net A2: now also JP1.11; no longer 328.11
- net A3: now also JP1.12; no longer 328.12
- net A4_SDA: now also JP1.13; no longer 328.13
- net A5_SCL: now also JP1.14; no longer 328.14
- net AREF: now also JP1.7; no longer 328.7
- net D0_RX: now also JP2.2; no longer LEFT.2
- net D10: now also H-BRIDGE.3-4EN, JP1.2; no longer 328.2
- net D11_MOSI: now also JP1.3; no longer 328.3
- net D12_MISO: now also JP1.4; no longer 328.4
- net D13: now also JP1.5; no longer 328.5
- net D1_TX: now also JP2.3; no longer LEFT.3
- net D2: now also JP2.4; no longer LEFT.4
- net D3: now also JP2.5; no longer LEFT.5
- net D4: now also JP2.6; no longer LEFT.6
- net D5: now also JP2.11; no longer LEFT.11
- net D6: now also JP2.12; no longer LEFT.12
- net D7: now also JP2.13; no longer LEFT.13
- net D8_CLK: now also JP2.14; no longer LEFT.14
- net D9: now also JP1.1; no longer 328.1, H-BRIDGE.3-4EN
- net GND: now also C5.2, JP1.8, JP2.8; no longer 328.8, LEFT.8
- net RESET: now also JP2.1; no longer LEFT.1
- net VCC: now also JP1.6, JP2.7, R10.1; no longer 328.6, LEFT.7
- net XTAL1: now also JP2.9; no longer LEFT.9
- net XTAL2: now also JP2.10; no longer LEFT.10
