File: furby/furby_osi.brd (EAGLE design)
At the start: 60 x 57.1 mm, 44 parts, among them IC1 ATMEGA168PROUND, IC2 74AC14N, J1 1X2-3.5MM

Commit message: FURBY
Parts:
- removed C1: 0.1uF, minimidi:C025-025X050
- removed C2: 100uF/6V, rcl-ez:E2,5-5
- removed C3, C4: (no value), adafruit:C025-025X050
- removed C5: (no value), adafruit:C050-025X075
- removed C6: 0.1uF, rcl-ez:C025-025X050
- removed C7: 100uF/16V, rcl-ez:E2,5-6
- removed D1: (no value), adafruit:DO-1N4148
- removed D5: (no value), diode:D-5
- removed H-BRIDGE: L293D, texas:DIL16
- removed IC2: 74AC14N, 74xx-eu:DIL14
- removed IC3: (no value), adafruit:TO92-INLINE
- removed J1: 1X2-3.5MM, adafruit:1X2-3.5MM
- removed JP3: (no value), SparkFun:1X02
- removed LOWER_MTR: (no value), adafruit_mod:JST-PH-2-THM
- removed R1, R14, R2, R3, R7, R8, R9: (no value), adafruit:0207/2V
- removed R10: 11.9k, adafruit:0204/7
- removed R11: 15.7k, adafruit:0204/7
- removed UPPER_MTR: (no value), SparkFun:MOLEX-1X2
- added JP5: (no value), SparkFun_mod:1X08
- added JP6: (no value), SparkFun:1X06
- moved I2C 52.4 mm to (56.7, 10.1)
- moved RESET 48.5 mm to (10.8, 6.22)
- moved R17 48.3 mm to (11.3, 13.4)
- moved JP1 41.0 mm to (50.8, 43.2), turned to 180 degrees
- moved C11 35.7 mm to (16.2, 15.2)
- moved JP2 30.9 mm to (17.8, 30.5), turned to 0 degrees
- moved U$3 23.7 mm to (48.1, 22.6), turned to 0 degrees
- moved R5 12.7 mm to (22.6, 24.3), turned to 0 degrees
- moved R4 11.3 mm to (22.9, 21.8), turned to 0 degrees
- moved IC1 8.12 mm to (34.3, 36.9), turned to 0 degrees
Connections:
- removed net N$1: H-BRIDGE.11, LOWER_MTR.2
- removed net N$22: H-BRIDGE.14, LOWER_MTR.1
- removed net N$24: C1.1, C3.1, D5.C, IC3.2
- removed net N$25: H-BRIDGE.3, UPPER_MTR.2
- removed net N$28: H-BRIDGE.6, UPPER_MTR.1
- removed net N$3: D1.A, JP3.2, R10.2, R11.1
- removed net N$4: C5.1, D1.C, IC2.13, JP3.1, R11.2
- removed net N$8: IC2.12
- removed net VCC: C2.+, C4.1, C6.1, ENCODE2.1, FTDI.4, H-BRIDGE.16, I2C.1, IC1.20, IC1.21, IC1.7, IC2.14, IC3.3, JP1.6, JP2.7, R10.1, R17.1
- new net +3V3: ENCODE2.1, IC1.20, IC1.21, JP6.4, R17.1
- new net +5V: JP5.7
- new net 3V3: FTDI.4, I2C.1, IC1.7, JP1.6, JP2.7
- new net A6: JP6.3
- new net A7: JP5.3
- new net M3A: JP5.2
- new net M4A: JP5.1
- new net N$5: UPPER.K
- new net N$6: LOWER.K
- net A2: now also JP6.1; no longer LOW_SW.1, R9.1
- net A3: now also JP6.2; no longer R3.1, UPPER_SW.1
- net D10: no longer H-BRIDGE.9
- net D11_MOSI: now also JP5.6; no longer H-BRIDGE.7, R2.2, UPPER.K
- net D12_MISO: now also JP5.5; no longer H-BRIDGE.2, R1.2
- net D13: now also JP5.4
- net D5: no longer H-BRIDGE.10, LOWER.K, R7.1
- net D7: no longer H-BRIDGE.15, R8.2
- net D9: no longer H-BRIDGE.1, R14.2
- net GND: now also JP6.5; no longer C1.2, C2.-, C3.2, C4.2, C5.2, C6.2, C7.-, H-BRIDGE.12, H-BRIDGE.13, H-BRIDGE.4, H-BRIDGE.5, IC2.7, IC3.1, J1.1, R1.1, R14.1, R2.1, R3.2, R7.2, R8.1, R9.2
- net RESET: now also JP6.6
- net V+: now also JP5.8; no longer C7.+, D5.A, H-BRIDGE.8, J1.2

Commit message: Furby work
Parts:
- removed R15, R17, R6: (no value), adafruit:0207/2V
- removed UPPER_SW: (no value), SparkFun:1X02
- added BATT: TERMINAL2, _my-parts:TERMINAL_2
- added D1: (no value), adafruit:DO-1N4148
- added JMP: (no value), SparkFun:1X02
- added JP3: (no value), SparkFun_mod:1X08
- added JP4: (no value), SparkFun:1X06
- added R1, R2, R3: (no value), adafruit:0204/7
- R4, R5: device SparkFun:1/6W-RES -> adafruit:0204/7
- moved I2C 49.4 mm to (10.8, 28.4), turned to 180 degrees
- moved RESET 43.4 mm to (13.8, 49.5), turned to 90 degrees
- moved C11 38.6 mm to (19.6, 53.6), turned to 0 degrees
- moved UPPER 6.39 mm to (29.1, 51.6), turned to 0 degrees
- moved LOWER 6.25 mm to (24.0, 51.6), turned to 0 degrees
- moved R5 3.37 mm to (24.1, 27.3)
- moved R4 3.19 mm to (24.1, 24.8)
- moved ENCODE1 1.91 mm to (36.1, 52.0)
- moved ENCODE2 1.91 mm to (40.1, 52.0)
- moved U$3 1.80 mm to (49.4, 21.3)
Connections:
- removed net +3V3: ENCODE2.1, IC1.20, IC1.21, JP6.4, R17.1
- removed net M3A: JP5.2
- removed net M4A: JP5.1
- removed net N$9: R15.1, UPPER.A
- new net N$1: R1.1, UPPER.A
- new net N$10: JP3.6
- new net N$11: JP3.7
- new net N$12: JP3.8
- new net N$15: JP4.3
- new net N$16: JP4.6
- new net N$3: BATT.P$2, JMP.2
- new net N$4: D1.A, JMP.1
- new net N$7: JP3.3
- net 3V3: now also D1.C, ENCODE2.1, IC1.20, IC1.21, JP4.4, JP6.4, R3.1, R4.2, R5.2
- net A0: now also JP6.2, UPPER.K
- net A1: now also JP6.1, R1.2
- net A2: now also JP5.1, R2.2; no longer JP6.1
- net A3: now also JP5.2, LOWER.K; no longer JP6.2
- net A6: now also JP5.3; no longer JP6.3
- net A7: now also JP6.3; no longer JP5.3
- net D12_MISO: no longer R15.2
- net D4: now also JP4.1
- net D5: now also JP3.5
- net D6: now also JP3.4
- net D7: now also JP4.2; no longer R6.1
- net GND: now also BATT.P$1, JP4.5; no longer R4.2, R5.2, UPPER_SW.2
- net N$2: now also R2.1; no longer R6.2
- net N$5: now also JP3.2; no longer UPPER.K
- net N$6: now also JP3.1; no longer LOWER.K
- net RESET: now also R3.2; no longer R17.2
Routing:
- net 3V3: track 0.00 -> 152.1 mm
- net RESET: track 0.00 -> 113.8 mm
- net D1_TX: track 0.00 -> 79.6 mm
- net RTS#: track 0.00 -> 62.3 mm
- net D6: track 0.00 -> 57.9 mm
- net D5: track 0.00 -> 56.1 mm
- net D7: track 0.00 -> 54.3 mm
- net D0_RX: track 0.00 -> 46.1 mm
- net D4: track 0.00 -> 41.5 mm, vias 0 -> 1
- net A5_SCL: track 0.00 -> 40.3 mm
- net A4_SDA: track 0.00 -> 34.1 mm
- net D2: track 0.00 -> 34.0 mm
- net D3: track 0.00 -> 33.9 mm
- net A1: track 0.00 -> 32.5 mm
- net A0: track 0.00 -> 27.3 mm
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Other:
- outline, holes or cut-outs redrawn
- board text added: "-POS -NEG"
- board text added: "10k"
- board text added: "330"
- board text added: "4.7k"
- board text added: "Batt"
- board text added: "Encoder"
- board text added: "Lower"
- board text added: "Reset"
- board text added: "Upper"
- board text removed: "L293D"
