File: furby/furby_osi.sch (EAGLE design)
At the start: 21 parts, among them IC1 ATMEGA168PROUND

Commit message: Furby work
Parts:
- removed R15, R17, R6: (no value), adafruit:R-US_0207/2V
- removed UPPER_SW: (no value), SparkFun:M02PTH
- added BATT: TERMINAL2, _my-parts:TERMINAL2
- added D1: (no value), adafruit:DIODEDO-1N4148
- added JMP: (no value), SparkFun:M02PTH
- added JP3: (no value), SparkFun_mod:M081X08
- added JP4: (no value), SparkFun:M06SIP
- added R1, R2, R3: (no value), adafruit:R-US_0204/7
- R4, R5: device SparkFun:RESISTORPTH-1/6W -> adafruit:R-US_0204/7
Connections:
- removed net +3V3: ENCODE2.2, IC1.AREF, IC1.AVCC, JP6.4, R17.1
- removed net M3A: JP5.2
- removed net M4A: JP5.1
- removed net N$9: R15.1, UPPER.A
- new net N$1: R1.1, UPPER.A
- new net N$10: JP3.6
- new net N$11: JP3.7
- new net N$12: JP3.8
- new net N$15: JP4.3
- new net N$16: JP4.6
- new net N$3: BATT.P$2, JMP.2
- new net N$4: D1.A, JMP.1
- new net N$7: JP3.3
- net 3V3: now also D1.C, ENCODE2.2, IC1.AREF, IC1.AVCC, JP4.4, JP6.4, R3.1, R4.2, R5.2
- net A0: now also JP6.2, UPPER.C
- net A1: now also JP6.1, R1.2
- net A2: now also JP5.1, R2.2; no longer JP6.1
- net A3: now also JP5.2, LOWER.C; no longer JP6.2
- net A6: now also JP5.3; no longer JP6.3
- net A7: now also JP6.3; no longer JP5.3
- net D12_MISO: no longer R15.2
- net D4: now also JP4.1
- net D5: now also JP3.5
- net D6: now also JP3.4
- net D7: now also JP4.2; no longer R6.1
- net GND: now also BATT.P$1, JP4.5; no longer R4.2, R5.2, UPPER_SW.2
- net N$2: now also R2.1; no longer R6.2
- net N$5: now also JP3.2; no longer UPPER.C
- net N$6: now also JP3.1; no longer LOWER.C
- net RESET: now also R3.2; no longer R17.2
Other:
- moved on the sheet: LOWER, UPPER
