File: osi/debounce/debounce_rev_2.brd (EAGLE design)
At the start: 25.4 x 25.4 mm, 33 parts, among them IC1 74LS14D

Commit message: Furby work
Parts:
- removed C5, C6: (no value), SparkFun:CAP-PTH-SMALL
- removed D5, D6: (no value), diode:D-2.5
- removed R10, R12: 15.7k, adafruit:0204V
- removed R11, R9: 11.9k, adafruit:0204V
- removed U$5, U$6: TERMINAL2, _my-parts:TERMINAL_2
- moved D4 81.9 mm to (22.6, 6.73), turned to 45 degrees
- moved R7 79.7 mm to (22.6, 13.7), turned to 45 degrees
- moved C4 77.2 mm to (23.5, 3.81), turned to 225 degrees
- moved R8 75.2 mm to (22.6, 10.0), turned to 225 degrees
- moved D3 4.07 mm to (19.7, 6.35), turned to 45 degrees
- moved R6 3.52 mm to (19.7, 9.91), turned to 225 degrees
- moved R5 3.24 mm to (19.7, 13.3), turned to 45 degrees
- moved C3 2.50 mm to (20.6, 4.06), turned to 225 degrees
- moved C2 1.44 mm to (7.24, 7.37), turned to 225 degrees
- moved R3 0.81 mm to (6.35, 13.5), turned to 45 degrees
- moved R4 0.68 mm to (6.35, 11.2), turned to 225 degrees
- moved D2 0.65 mm to (2.79, 8.64)
- moved D1 0.64 mm to (6.35, 8.89), turned to 45 degrees
- moved R1 0.64 mm to (2.79, 13.6)
- moved R2 0.64 mm to (2.79, 11.0)
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Connections:
- removed net +3V3: JP6.4
- removed net A6: JP6.3
- removed net A7: JP5.3
- removed net N$12: IC1.8
- removed net N$13: D5.A, R10.1, R9.2, U$5.P$1
- removed net N$14: C5.2, D5.C, IC1.11, R10.2, U$5.P$2
- removed net N$15: IC1.10
- removed net N$16: D6.A, R11.2, R12.1, U$6.P$1
- removed net N$17: C6.2, D6.C, IC1.13, R12.2, U$6.P$2
- removed net N$18: IC1.12
- removed net N$5: IC1.4
- removed net N$8: IC1.6
- removed net N$9: IC1.2
- net A2: now also IC1.6
- net A3: now also IC1.8
- net D12: now also IC1.4
- net D13: now also IC1.2
- net GND: now also JP5.3; no longer C5.1, C6.1
- net VCC: now also JP6.3, JP6.4; no longer R11.1, R9.1
Routing:
- net VCC: track 0.00 -> 65.9 mm
- net N$7: track 0.00 -> 26.6 mm
- net N$11: track 0.00 -> 24.0 mm
- net N$4: track 0.00 -> 23.5 mm
- net D12: track 0.00 -> 21.4 mm
- net D13: track 0.00 -> 19.2 mm
- net N$2: track 0.00 -> 18.0 mm
- net A2: track 0.00 -> 15.9 mm
- net A3: track 0.00 -> 13.1 mm
- net N$6: track 0.00 -> 12.6 mm
- net N$10: track 0.00 -> 11.4 mm
- net N$1: track 0.00 -> 10.1 mm
- net N$3: track 0.00 -> 9.19 mm
Other:
- board text added: "74HC14"
- board text added: "Debounce"
- board text removed: "Atmega328"
- board text removed: "NODE"
- board text removed: "i2c"
