File: furby/furby_shield/furby_shield_v1b.sch (EAGLE design)
At the start: 26 parts, among them IC1 UA7805CKCS, Q2 ZVNL110ASTZ, Q3 ZVNL110ASTZ

Commit message: furby updates
Parts:
- added C6: 47nF, rcl:C-EU025-030X050
- added C7: 100nF, rcl:C-EU025-025X050
- added C8, C9: 10uF, rcl:CPOL-EUE2.5-6
- added LM386: LM386N-1, linear:LM386N-1
- added R8, R9: (no value), adafruit:R-US_0204/7
Connections:
- removed net MIC_B: SENSORS.7
- new net A1: C6.1, LM386.OUT
- new net N$4: C6.2, R8.2
- new net N$6: C9.+, LM386.BYPASS
- new net N$8: C8.-, LM386.+IN
- net GND: now also C7.2, C9.-, LM386.-IN, LM386.GND, R8.1; no longer RESET.S1
- net MIC_A: now also C8.+, R9.1
- net RESET: no longer RESET.P1
- net VCC: now also C7.1, LM386.VS, R9.2
Other:
- note added: "- Original Design by: Dimitar Kovachev http://lowvoltage.wordpress.com"
- note added: "- Released under the Creative Commons Attribution Share-Alike 3.0 license"
- note added: "http://creativecommons.org/licenses/by-sa/3.0/"
Changed lines of the file:
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@@
 </variantdefs>
 <classes>
-<class number="0" name="default" width="0.2032" drill="0">
+<class number="0" name="default" width="0" drill="0">
 </class>
 <class number="1" name="power" width="0.6096" drill="0">
@@
 <part name="P+1" library="supply1" deviceset="+5V" device=""/>
 <part name="U1" library="SparkFun" deviceset="AUDIO-JACK" device="PTH"/>
+<part name="LM386" library="linear" deviceset="LM386?-*" device="N" technology="1" value=""/>
+<part name="C6" library="rcl" deviceset="C-EU" device="025-030X050" value="47nF"/>
+<part name="GND2" library="supply1" deviceset="GND" device=""/>
+<part name="GND8" library="supply1" deviceset="GND" device=""/>
+<part name="GND9" library="supply1" deviceset="GND" device=""/>
+<part name="GND10" library="supply1" deviceset="GND" device=""/>
+<part name="P+4" library="supply1" deviceset="VCC" device=""/>
+<part name="P+9" library="supply1" deviceset="VCC" device=""/>
+<part name="GND11" library="supply1" deviceset="GND" device=""/>
+<part name="C7" library="rcl" deviceset="C-EU" device="025-025X050" value="100nF"/>
+<part name="GND13" library="supply1" deviceset="GND" device=""/>
+<part name="P+11" library="supply1" deviceset="VCC" device=""/>
+<part name="C8" library="rcl" deviceset="CPOL-EU" device="E2.5-6" value="10uF"/>
+<part name="C9" library="rcl" deviceset="CPOL-EU" device="E2.5-6" value="10uF"/>
+<part name="R8" library="adafruit" deviceset="R-US_" device="0204/7"/>
+<part name="R9" library="adafruit" deviceset="R-US_" device="0204/7"/>
 </parts>
 <sheets>
@@
 <text x="147.32" y="27.94" size="2.54" layer="94">http://www.ladyada.net/make/mshield</text>
 <text x="10.16" y="7.62" size="1.27" layer="91">https://sites.google.com/site/fpgaandco/level-shifting-i2c</text>
+<text x="7.62" y="121.92" size="1.778" layer="97">- Original Design by: Dimitar Kovachev
+  http://lowvoltage.wordpress.com</text>
+<text x="7.62" y="129.54" size="1.778" layer="97">- Released under the Creative Commons Attribution
+  Share-Alike 3.0 license</text>
+<text x="7.62" y="127" size="1.778" layer="97">  http://creativecommons.org/licenses/by-sa/3.0/</text>
 </plain>
 <instances>
@@
 <instance part="P+1" gate="1" x="129.54" y="116.84"/>
 <instance part="U1" gate="G$1" x="93.98" y="50.8" rot="MR90"/>
+<instance part="LM386" gate="G$1" x="40.64" y="160.02" smashed="yes">
+<attribute name="NAME" x="53.34" y="157.48" size="1.778" layer="95" rot="R180"/>
+<attribute name="VALUE" x="45.72" y="156.21" size="1.778" layer="96"/>
+</instance>
+<instance part="C6" gate="G$1" x="53.34" y="157.48"/>
+<instance part="GND2" gate="1" x="33.02" y="139.7"/>
+<instance part="GND8" gate="1" x="38.1" y="139.7"/>
+<instance part="GND9" gate="1" x="43.18" y="139.7"/>
+<instance part="GND10" gate="1" x="53.34" y="139.7"/>
+<instance part="P+4" gate="VCC" x="38.1" y="175.26" smashed="yes">
+<attribute name="VALUE" x="40.64" y="177.8" size="1.778" layer="96" rot="R180"/>
+</instance>
+<instance part="P+9" gate="VCC" x="71.12" y="175.26" smashed="yes">
+<attribute name="VALUE" x="73.66" y="177.8" size="1.778" layer="96" rot="R180"/>
+</instance>
+<instance part="GND11" gate="1" x="71.12" y="139.7"/>
+<instance part="C7" gate="G$1" x="71.12" y="162.56"/>
+<instance part="GND13" gate="1" x="25.4" y="139.7"/>
+<instance part="P+11" gate="VCC" x="25.4" y="175.26" smashed="yes">
+<attribute name="VALUE" x="27.94" y="177.8" size="1.778" layer="96" rot="R180"/>
+</instance>
+<instance part="C8" gate="G$1" x="27.94" y="162.56" smashed="yes" rot="R90">
+<attribute name="NAME" x="30.607" y="167.1574" size="1.778" layer="95" rot="R180"/>
+<attribute name="VALUE" x="33.147" y="159.5374" size="1.778" layer="96" rot="R180"/>
+</instance>
+<instance part="C9" gate="G$1" x="43.18" y="149.86" smashed="yes">
+<attribute name="NAME" x="47.7774" y="147.193" size="1.778" layer="95" rot="R90"/>
+<attribute name="VALUE" x="40.1574" y="144.653" size="1.778" layer="96" rot="R90"/>
+</instance>
+<instance part="R8" gate="G$1" x="53.34" y="147.32" rot="R90"/>
+<instance part="R9" gate="G$1" x="25.4" y="167.64" rot="R90"/>
 </instances>
 <busses>
@@
 </segment>
 <segment>
-<wire x1="-43.18" y1="78.74" x2="-45.72" y2="78.74" width="0.1524" layer="91"/>
-<junction x="-43.18" y="78.74"/>
-<junction x="-45.72" y="78.74"/>
 <pinref part="RESET" gate="1" pin="S"/>
-<pinref part="RESET" gate="1" pin="S1"/>
 <pinref part="GND5" gate="1" pin="GND"/>
 </segment>
@@
 <pinref part="MOTORS" gate="G$1" pin="9"/>
 </segment>
+<segment>
+<wire x1="43.18" y1="142.24" x2="43.18" y2="144.78" width="0.1524" layer="91"/>
+<pinref part="GND9" gate="1" pin="GND"/>
+<pinref part="C9" gate="G$1" pin="-"/>
+</segment>
+<segment>
+<wire x1="38.1" y1="142.24" x2="38.1" y2="152.4" width="0.1524" layer="91"/>
+<pinref part="GND8" gate="1" pin="GND"/>
+<pinref part="LM386" gate="G$1" pin="GND"/>
+</segment>
+<segment>
+<wire x1="71.12" y1="142.24" x2="71.12" y2="157.48" width="0.1524" layer="91"/>
+<pinref part="GND11" gate="1" pin="GND"/>
+<pinref part="C7" gate="G$1" pin="2"/>
+</segment>
+<segment>
+<wire x1="33.02" y1="157.48" x2="33.02" y2="142.24" width="0.1524" layer="91"/>
+<pinref part="LM386" gate="G$1" pin="-IN"/>
+<pinref part="GND2" gate="1" pin="GND"/>
+</segment>
+<segment>
+<pinref part="GND10" gate="1" pin="GND"/>
+<pinref part="R8" gate="G$1" pin="1"/>
+</segment>
 </net>
 <net name="RESET" class="0">
 <segment>
 <wire x1="-45.72" y1="101.6" x2="-45.72" y2="88.9" width="0.1524" layer="91"/>
-<wire x1="-45.72" y1="88.9" x2="-43.18" y2="88.9" width="0.1524" layer="91"/>
-<junction x="-43.18" y="88.9"/>
-<junction x="-45.72" y="88.9"/>
 <label x="-45.72" y="93.98" size="1.778" layer="95" rot="R90"/>
-<pinref part="RESET" gate="1" pin="P1"/>
 <pinref part="RESET" gate="1" pin="P"/>
 <pinref part="U$1" gate="G$1" pin="/RESET"/>
@@
 <wire x1="55.88" y1="27.94" x2="60.96" y2="27.94" width="0.1524" layer="91"/>
 <junction x="55.88" y="27.94"/>
+</segment>
+<segment>
+<wire x1="38.1" y1="167.64" x2="38.1" y2="172.72" width="0.1524" layer="91"/>
+<pinref part="LM386" gate="G$1" pin="VS"/>
+<pinref part="P+4" gate="VCC" pin="VCC"/>
+</segment>
+<segment>
+<wire x1="71.12" y1="165.1" x2="71.12" y2="172.72" width="0.1524" layer="91"/>
+<pinref part="C7" gate="G$1" pin="1"/>
+<pinref part="P+9" gate="VCC" pin="VCC"/>
+</segment>
+<segment>
+<pinref part="P+11" gate="VCC" pin="VCC"/>
+<pinref part="R9" gate="G$1" pin="2"/>
 </segment>
 </net>
@@
 <label x="-25.4" y="93.98" size="1.778" layer="95" rot="R90"/>
 </segment>
+<segment>
+<wire x1="25.4" y1="162.56" x2="22.86" y2="162.56" width="0.1524" layer="91"/>
+<pinref part="C8" gate="G$1" pin="+"/>
+<label x="15.24" y="162.56" size="1.778" layer="95"/>
+<pinref part="R9" gate="G$1" pin="1"/>
+<junction x="25.4" y="162.56"/>
+</segment>
 </net>
 <net name="MIC_B" class="0">
 <segment>
-<wire x1="101.6" y1="86.36" x2="101.6" y2="96.52" width="0.1524" layer="91"/>
-<label x="101.6" y="86.36" size="1.778" layer="95" rot="R90"/>
-<pinref part="SENSORS" gate="G$1" pin="7"/>
+<wire x1="25.4" y1="160.02" x2="25.4" y2="142.24" width="0.1524" layer="91"/>
+<wire x1="22.86" y1="160.02" x2="25.4" y2="160.02" width="0.1524" layer="91"/>
+<pinref part="GND13" gate="1" pin="GND"/>
+<label x="15.24" y="160.02" size="1.778" layer="95"/>
 </segment>
 </net>
@@
 </segment>
 </net>
+<net name="A1" class="0">
+<segment>
+<wire x1="50.8" y1="160.02" x2="53.34" y2="160.02" width="0.1524" layer="91"/>
+<wire x1="53.34" y1="160.02" x2="58.42" y2="160.02" width="0.1524" layer="91"/>
+<junction x="53.34" y="160.02"/>
+<pinref part="C6" gate="G$1" pin="1"/>
+<pinref part="LM386" gate="G$1" pin="OUT"/>
+<label x="55.88" y="160.02" size="1.778" layer="95"/>
+</segment>
+</net>
+<net name="N$6" class="0">
+<segment>
+<wire x1="43.18" y1="152.4" x2="43.18" y2="154.94" width="0.1524" layer="91"/>
+<pinref part="LM386" gate="G$1" pin="BYPASS"/>
+<pinref part="C9" gate="G$1" pin="+"/>
+</segment>
+</net>
+<net name="N$8" class="0">
+<segment>
+<pinref part="C8" gate="G$1" pin="-"/>
+<pinref part="LM386" gate="G$1" pin="+IN"/>
+</segment>
+</net>
+<net name="N$4" class="0">
+<segment>
+<pinref part="C6" gate="G$1" pin="2"/>
+<pinref part="R8" gate="G$1" pin="2"/>
+</segment>
+</net>
 </nets>
 </sheet>
@@
 </schematic>
 </drawing>
+<compatibility>
+<note version="6.3" minversion="6.2.2" severity="warning">
+Since Version 6.2.2 text objects can contain more than one line,
+which will not be processed correctly with this version.
+</note>
+</compatibility>
 </eagle>

Commit message: furby board production
Parts:
- removed TRACKS: L293D, texas:L293E
- added L293D: (no value), texas:L293E
- R8, R9: value (none) -> 10k
Connections:
- net +5V: now also L293D.VCC1, L293D.VCC2; no longer TRACKS.VCC1, TRACKS.VCC2
- net D12: now also L293D.3-4EN; no longer TRACKS.3-4EN
- net D13: now also L293D.1-2EN; no longer TRACKS.1-2EN
- net GND: now also L293D.GND1, L293D.GND2, L293D.GND3, L293D.GND4; no longer TRACKS.GND1, TRACKS.GND2, TRACKS.GND3, TRACKS.GND4
- net LM1: now also L293D.3A; no longer TRACKS.3A
- net LM2: now also L293D.4A; no longer TRACKS.4A
- net L_MTR_1: now also L293D.4Y; no longer TRACKS.4Y
- net L_MTR_2: now also L293D.3Y; no longer TRACKS.3Y
- net UM1: now also L293D.2A; no longer TRACKS.2A
- net UM2: now also L293D.1A; no longer TRACKS.1A
- net U_MTR_1: now also L293D.1Y; no longer TRACKS.1Y
- net U_MTR_2: now also L293D.2Y; no longer TRACKS.2Y
Other:
- moved on the sheet: C1, C2, C3, C4, C5, C6, C7, C8, C9, IC1, LED1, LED2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
