File: furby/furby_shield/furby_shield_v1b.brd (EAGLE design)
At the start: 68.6 x 53.3 mm, 26 parts, among them IC1 UA7805CKCS, Q2 ZVNL110ASTZ, Q3 ZVNL110ASTZ

Commit message: furby updates
Parts:
- added C6: 47nF, rcl:C025-030X050
- added C7: 100nF, rcl:C025-025X050
- added C8, C9: 10uF, rcl:E2,5-6
- added LM386: (no value), linear:DIL08
- added R8, R9: (no value), adafruit:0204/7
- moved LED2 24.3 mm to (64.8, 26.0)
- moved LED3 22.9 mm to (64.8, 33.7)
- moved R6 20.4 mm to (64.8, 29.8), turned to 180 degrees
- moved R7 17.1 mm to (64.8, 37.5), turned to 180 degrees
- moved C5 11.4 mm to (44.5, 36.8), turned to 180 degrees
- moved R1 11.4 mm to (64.9, 22.2)
- moved LED1 10.2 mm to (64.8, 18.4)
- moved C1 9.09 mm to (37.5, 33.7), turned to 90 degrees
- moved TRACKS 8.82 mm to (50.8, 29.8)
- moved SENSORS 8.26 mm to (33.0, 43.8)
- moved C4 6.87 mm to (51.4, 18.4), turned to 90 degrees
- moved C2 6.54 mm to (59.7, 18.4), turned to 180 degrees
- moved C3 5.99 mm to (55.2, 18.4), turned to 90 degrees
- moved MOTORS 4.96 mm to (55.9, 43.8)
- moved RESET 1.78 mm to (22.6, 4.83), turned to 180 degrees
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Connections:
- removed net MIC_B: SENSORS.7
- new net A1: C6.1, LM386.5
- new net N$4: C6.2, R8.2
- new net N$6: C9.+, LM386.7
- new net N$8: C8.-, LM386.3
- net GND: now also C7.2, C9.-, LM386.2, LM386.4, R8.1; no longer RESET.2
- net MIC_A: now also C8.+, R9.1
- net RESET: no longer RESET.4
- net VCC: now also C7.1, LM386.6, R9.2
Routing:
- net +5V: track 100.8 -> 71.9 mm
- net UM1: track 50.8 -> 24.2 mm
- net D12: track 56.3 -> 47.0 mm
- net PIEZO: track 18.5 -> 9.89 mm
- net LM2: track 25.5 -> 17.8 mm, vias 1 -> 0
- net LEVEL_A: track 58.3 -> 50.8 mm
- net BEAK: track 27.6 -> 20.6 mm
- net SPR_B: track 26.3 -> 32.6 mm
- net L_MTR_1: track 31.1 -> 36.9 mm
- net BELLY: track 21.5 -> 15.8 mm
- net LM1: track 32.0 -> 26.4 mm
- net SPR_A: track 24.5 -> 30.0 mm
- net RESET: track 14.9 -> 9.43 mm
- net VCC: track 86.7 -> 81.3 mm
- net N$8: track 0.00 -> 5.23 mm
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
Commit message: furby board production
Parts:
- added U$2: (no value), adafruit:OSHWLOGO_TOP_0.2
- L293D: value L293D -> (none)
- R8, R9: value (none) -> 10k
- moved RESET 1.33 mm to (22.2, 6.10)
- turned C1 to 180 degrees
- renumbered TRACKS to L293D
Routing:
- net +5V: track 71.9 -> 70.1 mm
- net RESET: track 9.43 -> 10.7 mm
- net +3V3: track 52.2 -> 51.5 mm
Other:
- board text added: "100nF"
- board text added: "10uF"
- board text added: "47nF"
- board text added: "Designed and Manufactured in OREGON"
- board text added: "Furby Shield"
- board text added: "Furby Shield Rev 0 Apr '13"
- board text added: "LM386"
- board text added: "MakersBox.blogspot.com"
- board text added: "Open Source Hardware"

Commit message: Joule Thief V5
Parts:
- added U$3: (no value), _my-parts:OREGON_18_51
- added U$4: (no value), _my-parts:OREGON_18_52
Other:
- board text added: "Furby Shield Rev 0 May '13"
- board text removed: "Furby Shield Rev 0 Apr '13"
Changed lines of the file:
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@@
 <setting verticaltext="up"/>
 </settings>
-<grid distance="0.05" unitdist="inch" unit="inch" style="lines" multiple="1" display="yes" altdistance="0.005" altunitdist="inch" altunit="inch"/>
+<grid distance="0.01" unitdist="inch" unit="inch" style="lines" multiple="1" display="yes" altdistance="0.005" altunitdist="inch" altunit="inch"/>
 <layers>
 <layer number="1" name="Top" color="4" fill="1" visible="yes" active="yes"/>
@@
 <layer number="27" name="tValues" color="7" fill="1" visible="no" active="yes"/>
 <layer number="28" name="bValues" color="7" fill="1" visible="no" active="yes"/>
-<layer number="29" name="tStop" color="7" fill="3" visible="no" active="yes"/>
+<layer number="29" name="tStop" color="7" fill="3" visible="yes" active="yes"/>
 <layer number="30" name="bStop" color="7" fill="6" visible="no" active="yes"/>
-<layer number="31" name="tCream" color="7" fill="4" visible="no" active="yes"/>
+<layer number="31" name="tCream" color="7" fill="4" visible="yes" active="yes"/>
 <layer number="32" name="bCream" color="7" fill="5" visible="no" active="yes"/>
 <layer number="33" name="tFinish" color="6" fill="3" visible="no" active="yes"/>
@@
 <layer number="50" name="dxf" color="7" fill="1" visible="no" active="yes"/>
 <layer number="51" name="tDocu" color="6" fill="1" visible="yes" active="yes"/>
-<layer number="52" name="bDocu" color="7" fill="1" visible="no" active="yes"/>
+<layer number="52" name="bDocu" color="7" fill="1" visible="yes" active="yes"/>
 <layer number="53" name="tGND_GNDA" color="7" fill="9" visible="no" active="no"/>
 <layer number="54" name="bGND_GNDA" color="1" fill="9" visible="no" active="no"/>
@@
 <wire x1="0.381" y1="0" x2="0.381" y2="14.732" width="0" layer="20"/>
 <wire x1="0.381" y1="29.9085" x2="0.381" y2="53.34" width="0" layer="20"/>
-<rectangle x1="53.086" y1="5.715" x2="69.088" y2="17.018" layer="29"/>
-<rectangle x1="53.086" y1="5.715" x2="69.088" y2="17.018" layer="31"/>
 <text x="47.498" y="29.083" size="1.778" layer="21" font="vector" ratio="15">L293D</text>
 <text x="18.796" y="0.635" size="1.778" layer="21" font="vector" ratio="15">Reset</text>
@@
 <text x="8.89" y="29.21" size="1.4224" layer="21" font="vector" ratio="15">I2C</text>
 <text x="25.146" y="13.716" size="1.4224" layer="21" font="vector" ratio="12" rot="R90">Level Shifting</text>
-<text x="46.863" y="32.512" size="1.016" layer="21" font="vector" ratio="10">330</text>
+<text x="63.627" y="21.717" size="1.016" layer="21" font="vector" ratio="10">330</text>
 <text x="63.373" y="36.957" size="1.016" layer="21" font="vector" ratio="10">330</text>
 <text x="66.929" y="36.449" size="1.4224" layer="21" font="vector" ratio="12" rot="R270">Legs</text>
@@
 <text x="26.67" y="32.385" size="1.778" layer="52" font="vector" ratio="15" rot="MR0">Furby Shield
 Rev 0
-Apr '13</text>
+May '13</text>
 <text x="64.516" y="47.371" size="1.778" layer="52" font="vector" ratio="15" rot="MR0">MakersBox.blogspot.com</text>
 <text x="15.24" y="3.81" size="1.27" layer="52" font="vector" ratio="10" rot="MR0">Designed and
 Manufactured
  in OREGON</text>
+<rectangle x1="53.34" y1="4.826" x2="69.088" y2="15.494" layer="29"/>
+<rectangle x1="53.34" y1="4.826" x2="69.088" y2="15.494" layer="31"/>
 </plain>
 <attributes>
@@
 <element name="R9" library="adafruit" package="0204/7" value="10k" x="42.545" y="17.145" rot="R270"/>
 <element name="U$2" library="adafruit" package="OSHWLOGO_TOP_0.2" value="" x="18.415" y="41.275"/>
+<element name="U$3" library="_my-parts" package="OREGON_18_51" value="" x="41.275" y="11.176"/>
+<element name="U$4" library="_my-parts" package="OREGON_18_52" value="" x="46.99" y="11.43"/>
 </elements>
 <signals>
