File: osi/ftdi/ftdi_rev_3.brd (EAGLE design)
At the start: 24.8 x 25.4 mm, 4 parts

Commit message: double board finished?
Parts:
- added U$1: (no value), _my-parts:OREGON_18_52
Routing:
- net TXO: track 0.00 -> 19.6 mm
- net DTR: track 0.00 -> 15.0 mm
- net RXI: track 0.00 -> 14.5 mm
- net +3V3: track 0.00 -> 12.9 mm
Other:
- board text added: "FTDI"
- board text added: "May 13"
- board text removed: "3V"
- board text removed: "Apr 12"
- board text removed: "Atmega328"
- board text removed: "NODE"
- board text removed: "RST"
- board text removed: "i2c"
Changed lines of the file:
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@@
 <setting verticaltext="up"/>
 </settings>
-<grid distance="0.05" unitdist="inch" unit="inch" style="lines" multiple="1" display="yes" altdistance="0.005" altunitdist="inch" altunit="inch"/>
+<grid distance="0.025" unitdist="inch" unit="inch" style="lines" multiple="1" display="yes" altdistance="0.005" altunitdist="inch" altunit="inch"/>
 <layers>
 <layer number="1" name="Top" color="4" fill="1" visible="yes" active="yes"/>
@@
 <layer number="50" name="dxf" color="7" fill="1" visible="no" active="no"/>
 <layer number="51" name="tDocu" color="6" fill="1" visible="yes" active="yes"/>
-<layer number="52" name="bDocu" color="7" fill="1" visible="no" active="yes"/>
+<layer number="52" name="bDocu" color="7" fill="1" visible="yes" active="yes"/>
 <layer number="53" name="tGND_GNDA" color="7" fill="9" visible="no" active="no"/>
 <layer number="54" name="bGND_GNDA" color="1" fill="9" visible="no" active="no"/>
@@
 <wire x1="0.000159375" y1="21.590159375" x2="0" y2="21.590159375" width="0" layer="20"/>
 <wire x1="0" y1="21.590159375" x2="0" y2="0" width="0" layer="20"/>
-<text x="42.799" y="7.62" size="0.8128" layer="21" font="vector" ratio="15" rot="R180">Atmega328</text>
-<text x="36.068" y="19.812" size="2.1844" layer="21" font="vector" ratio="20" rot="R270">NODE</text>
-<text x="51.308" y="1.016" size="1.016" layer="22" font="vector" ratio="15" rot="SMR0">MakersBox.blogspot.com</text>
-<text x="33.528" y="3.175" size="1.016" layer="22" font="vector" ratio="12" rot="MR0">Apr 12</text>
+<text x="15.113" y="6.223" size="2.1844" layer="21" font="vector" ratio="20">FTDI</text>
+<text x="23.241" y="0.762" size="1.016" layer="22" font="vector" ratio="15" rot="SMR90">MakersBox.blogspot.com</text>
+<text x="22.098" y="3.81" size="1.016" layer="22" font="vector" ratio="12" rot="MR0">May 13</text>
 <text x="22.86" y="21.717" size="1.016" layer="21" font="vector" ratio="15">V+</text>
-<text x="11.684" y="2.794" size="0.8128" layer="21" font="vector" ratio="15">GND</text>
 <text x="20.32" y="21.717" size="1.016" layer="21" font="vector" ratio="15">5V</text>
-<text x="9.398" y="2.794" size="1.016" layer="21" font="vector" ratio="15">3V</text>
-<text x="14.351" y="2.794" size="0.8128" layer="21" font="vector" ratio="15">RST</text>
 <text x="22.479" y="22.479" size="1.016" layer="22" font="vector" ratio="15" rot="MR180">V+</text>
 <text x="19.812" y="22.479" size="1.016" layer="22" font="vector" ratio="15" rot="MR180">5V</text>
@@
 <text x="14.224" y="22.606" size="1.016" layer="22" font="vector" ratio="15" rot="MR180">A2</text>
 <text x="18.542" y="21.59" size="1.016" layer="22" font="vector" ratio="15" rot="MR0">DTR</text>
-<text x="41.148" y="3.048" size="2.1844" layer="22" ratio="12" rot="SMR0">NODE</text>
+<text x="22.098" y="6.223" size="2.1844" layer="22" ratio="12" rot="SMR0">FTDI</text>
 <text x="6.858" y="2.794" size="1.016" layer="21" font="vector" ratio="15">D4</text>
 <text x="4.318" y="2.794" size="1.016" layer="21" font="vector" ratio="15">D3</text>
@@
 <text x="4.318" y="21.717" size="1.016" layer="21" font="vector" ratio="15">P1</text>
 <text x="12.319" y="21.717" size="1.016" layer="21" font="vector" ratio="15">A1</text>
-<text x="45.974" y="23.876" size="0.8128" layer="21" font="vector" ratio="10" rot="R180">MakersBox.blogspot.com</text>
+<text x="23.114" y="19.304" size="1.016" layer="21" font="vector" ratio="10" rot="R270">MakersBox.blogspot.com</text>
 <text x="11.684" y="22.606" size="1.016" layer="22" font="vector" ratio="15" rot="MR180">A1</text>
 <text x="3.175" y="2.794" size="1.016" layer="22" font="vector" ratio="15" rot="MR0">D2</text>
 <text x="5.969" y="2.794" size="1.016" layer="22" font="vector" ratio="15" rot="MR0">D3</text>
 <text x="8.382" y="2.794" size="1.016" layer="22" font="vector" ratio="15" rot="MR0">D4</text>
-<text x="10.922" y="2.794" size="1.016" layer="22" font="vector" ratio="15" rot="MR0">3V</text>
-<text x="13.716" y="2.794" size="0.8128" layer="22" font="vector" ratio="15" rot="MR0">GND</text>
-<text x="16.383" y="2.794" size="0.8128" layer="22" font="vector" ratio="15" rot="SMR0">RST</text>
-<text x="34.036" y="10.541" size="1.016" layer="22" font="vector" ratio="15" rot="MR270">i2c</text>
 <text x="8.128" y="18.542" size="1.27" layer="21" font="vector" ratio="12">DTR</text>
 <text x="8.128" y="16.002" size="1.27" layer="21" font="vector" ratio="12">TXo</text>
@@
 <element name="JP2" library="SparkFun_mod" package="1X06" value="" x="6.35" y="19.05" rot="R270"/>
 <element name="JP1" library="SparkFun_mod" package="1X02" value="" x="13.97" y="3.81" rot="R180"/>
+<element name="U$1" library="_my-parts" package="OREGON_18_52" value="" x="20.955" y="19.05"/>
 </elements>
 <signals>
@@
 <contactref element="JP2" pad="5"/>
 <contactref element="JP2" pad="6"/>
-<wire x1="6.35" y1="6.35" x2="12.7" y2="1.27" width="0" layer="19" extent="1-1"/>
-<wire x1="6.35" y1="8.89" x2="6.35" y2="6.35" width="0" layer="19" extent="1-1"/>
 </signal>
 <signal name="RESET">
@@
 <contactref element="JP6" pad="4"/>
 <contactref element="JP2" pad="4"/>
-<wire x1="6.35" y1="11.43" x2="10.16" y2="1.27" width="0" layer="19" extent="1-1"/>
+<wire x1="10.16" y1="1.27" x2="10.16" y2="1.905" width="0.4064" layer="16"/>
+<wire x1="10.16" y1="1.905" x2="9.525" y2="2.54" width="0.4064" layer="16"/>
+<wire x1="9.525" y1="2.54" x2="9.525" y2="10.16" width="0.4064" layer="16"/>
+<wire x1="9.525" y1="10.16" x2="8.255" y2="11.43" width="0.4064" layer="16"/>
+<wire x1="8.255" y1="11.43" x2="6.35" y2="11.43" width="0.4064" layer="16"/>
 </signal>
 <signal name="+5V">
@@
 <contactref element="JP2" pad="2"/>
 <contactref element="JP1" pad="1"/>
-<wire x1="13.97" y1="3.81" x2="6.35" y2="16.51" width="0" layer="19" extent="1-1"/>
+<wire x1="13.97" y1="3.81" x2="13.97" y2="15.24" width="0.4064" layer="16"/>
+<wire x1="13.97" y1="15.24" x2="12.7" y2="16.51" width="0.4064" layer="16"/>
+<wire x1="12.7" y1="16.51" x2="6.35" y2="16.51" width="0.4064" layer="16"/>
 </signal>
 <signal name="RXI">
 <contactref element="JP2" pad="3"/>
 <contactref element="JP1" pad="2"/>
-<wire x1="11.43" y1="3.81" x2="6.35" y2="13.97" width="0" layer="19" extent="1-1"/>
+<wire x1="11.43" y1="3.81" x2="11.43" y2="12.7" width="0.4064" layer="16"/>
+<wire x1="11.43" y1="12.7" x2="10.16" y2="13.97" width="0.4064" layer="16"/>
+<wire x1="10.16" y1="13.97" x2="6.35" y2="13.97" width="0.4064" layer="16"/>
 </signal>
 <signal name="DTR">
 <contactref element="JP2" pad="1"/>
 <contactref element="JP5" pad="6"/>
-<wire x1="6.35" y1="19.05" x2="17.78" y2="24.13" width="0" layer="19" extent="1-1"/>
+<wire x1="17.78" y1="24.13" x2="17.78" y2="21.59" width="0.4064" layer="16"/>
+<wire x1="17.78" y1="21.59" x2="15.24" y2="19.05" width="0.4064" layer="16"/>
+<wire x1="15.24" y1="19.05" x2="6.35" y2="19.05" width="0.4064" layer="16"/>
 </signal>
 </signals>
