File: JouleThief/joule_thief_v5.sch (EAGLE design)
At the start: 12 parts

Commit message: Joule Thief V5
Connections:
- net N$7: now also JP3.1
Changed lines of the file:
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@@
 <wire x1="50.8" y1="121.92" x2="22.86" y2="121.92" width="0.1524" layer="91"/>
 <junction x="50.8" y="121.92"/>
+<pinref part="JP3" gate="G$1" pin="1"/>
+<wire x1="22.86" y1="132.08" x2="22.86" y2="137.16" width="0.1524" layer="91"/>
+<junction x="22.86" y="132.08"/>
 </segment>
 </net>
